File: PAC5523/PAC5523.sch (KiCad schematic (older format))
At the start: 68 parts, among them J1 W, J2 U, J3 V, Q1 AON6276, U1 PAC5523, U10 PA1137NL

Commit message: wip
Parts:
- removed X?: ASCO, Oscillator:Oscillator_SMD_Abracon_ASCO-4Pin_1.6x1.2mm, symbol Oscillator:ASCO
- added C41: 18p, Capacitor_SMD:C_0603_1608Metric, symbol Device:C_Small
- added U4: Oscillator_3225, otter:Oscillator_3225, symbol otter:Oscillator_3225
Connections:
- net CLK: now also C41.1, U4.3 (OUT)
- net GND: now also C41.2, U4.2 (GND)
- net VIO: now also U4.4 (VCC)
Other:
- note removed: "TVS Diode\nWiderstand"
- note removed: "Todo:\nOszillator\n"
Changed lines of the file:
@@
 Text GLabel 1650 3850 0    50   Input ~ 0
 IUH
-Text Notes 3700 1200 0    50   ~ 0
-Todo:\nOszillator\n
 $Comp
 L Connector:Conn_01x06_Male J2
@@
 F1 "IC.sch" 50
 $EndSheet
-Text Notes 5100 1550 0    50   ~ 0
-TVS Diode\nWiderstand
 Wire Wire Line
 	10650 3400 10200 3400
@@
 Text GLabel 2300 2000 1    50   Input ~ 0
 NTC_IO
-$Comp
-L Oscillator:ASCO X?
-U 1 1 5CE0A013
-P 2000 5650
-F 0 "X?" H 2450 5750 50  0000 L CNN
-F 1 "ASCO" H 2450 5550 50  0000 L CNN
-F 2 "Oscillator:Oscillator_SMD_Abracon_ASCO-4Pin_1.6x1.2mm" H 2100 5300 50  0001 C CNN
-F 3 "https://abracon.com/Oscillators/ASCO.pdf" H 1775 5775 50  0001 C CNN
-	1    2000 5650
-	1    0    0    -1
-$EndComp
-Text GLabel 2400 5650 2    50   Input ~ 0
+Text GLabel 2650 5550 2    50   Input ~ 0
 CLK
-Text GLabel 2000 5350 1    50   Input ~ 0
+Text GLabel 1600 5550 0    50   Input ~ 0
 VIO
 $Comp
-L power:GND #PWR?
+L power:GND #PWR0162
 U 1 1 5CE19C05
-P 2000 5950
-F 0 "#PWR?" H 2000 5700 50  0001 C CNN
-F 1 "GND" H 2005 5777 50  0000 C CNN
-F 2 "" H 2000 5950 50  0001 C CNN
-F 3 "" H 2000 5950 50  0001 C CNN
-	1    2000 5950
-	1    0    0    -1
-$EndComp
-NoConn ~ 1600 5650
+P 1600 5750
+F 0 "#PWR0162" H 1600 5500 50  0001 C CNN
+F 1 "GND" H 1605 5577 50  0000 C CNN
+F 2 "" H 1600 5750 50  0001 C CNN
+F 3 "" H 1600 5750 50  0001 C CNN
+	1    1600 5750
+	0    1    1    0
+$EndComp
+NoConn ~ 2200 5750
+$Comp
+L otter:Oscillator_3225 U4
+U 1 1 5CDC2B99
+P 1900 5650
+F 0 "U4" H 1900 5975 50  0000 C CNN
+F 1 "Oscillator_3225" H 1900 5884 50  0000 C CNN
+F 2 "otter:Oscillator_3225" H 1900 6050 50  0001 C CNN
+F 3 "" H 1900 6050 50  0001 C CNN
+	1    1900 5650
+	1    0    0    -1
+$EndComp
+$Comp
+L Device:C_Small C41
+U 1 1 5CDC3C4D
+P 2400 5650
+F 0 "C41" H 2492 5696 50  0000 L CNN
+F 1 "18p" H 2492 5605 50  0000 L CNN
+F 2 "Capacitor_SMD:C_0603_1608Metric" H 2400 5650 50  0001 C CNN
+F 3 "~" H 2400 5650 50  0001 C CNN
+	1    2400 5650
+	1    0    0    -1
+$EndComp
+$Comp
+L power:GND #PWR0163
+U 1 1 5CDC3C53
+P 2400 5750
+F 0 "#PWR0163" H 2400 5500 50  0001 C CNN
+F 1 "GND" H 2405 5577 50  0000 C CNN
+F 2 "" H 2400 5750 50  0001 C CNN
+F 3 "" H 2400 5750 50  0001 C CNN
+	1    2400 5750
+	1    0    0    -1
+$EndComp
+Wire Wire Line
+	2650 5550 2400 5550
+Connection ~ 2400 5550
+Wire Wire Line
+	2400 5550 2200 5550
 $EndSCHEMATC

Commit message: placement almost done
Parts:
- R1: footprint Resistor_SMD:R_0805_2012Metric -> Resistor_SMD:R_0603_1608Metric
Connections:
- net +5V: now also C24.1
- net VIO: no longer C24.1
Changed lines of the file:
@@
 F 0 "R1" V 9054 1500 50  0000 C CNN
 F 1 "TBD" V 9145 1500 50  0000 C CNN
-F 2 "Resistor_SMD:R_0805_2012Metric" H 9250 1500 50  0001 C CNN
+F 2 "Resistor_SMD:R_0603_1608Metric" H 9250 1500 50  0001 C CNN
 F 3 "~" H 9250 1500 50  0001 C CNN
 	1    9250 1500
@@
 	1    0    0    -1
 $EndComp
-Text GLabel 6300 4850 1    50   Input ~ 0
-VIO
 $Comp
 L power:GND #PWR0116
@@
 Wire Wire Line
 	2400 5550 2200 5550
+$Comp
+L power:+5V #PWR?
+U 1 1 5CE806B5
+P 6300 4850
+AR Path="/5D5C3A79/5CE806B5" Ref="#PWR?"  Part="1"
+AR Path="/5CE806B5" Ref="#PWR0190"  Part="1"
+F 0 "#PWR0190" H 6300 4700 50  0001 C CNN
+F 1 "+5V" V 6315 4978 50  0000 L CNN
+F 2 "" H 6300 4850 50  0001 C CNN
+F 3 "" H 6300 4850 50  0001 C CNN
+	1    6300 4850
+	1    0    0    -1
+$EndComp
 $EndSCHEMATC

Commit message: routing 60% done
Connections:
- net GNDPWR is gone; now on net GND: C20.2, C21.2, C22.2, C23.2, C25.2, C33.2, R14.2, U10.10, U10.9
Changed lines of the file:
@@
 IWH
-$Comp
-L power:GNDPWR #PWR0118
-U 1 1 5CD65993
-P 6250 1300
-F 0 "#PWR0118" H 6250 1100 50  0001 C CNN
-F 1 "GNDPWR" H 6171 1273 50  0000 R CNN
-F 2 "" H 6250 1250 50  0001 C CNN
-F 3 "" H 6250 1250 50  0001 C CNN
-	1    6250 1300
-	1    0    0    -1
-$EndComp
 $Comp
 L Device:D_Small D15
@@
 $EndComp
 $Comp
-L power:GNDPWR #PWR0119
-U 1 1 5CD7AE42
-P 7000 1850
-F 0 "#PWR0119" H 7000 1650 50  0001 C CNN
-F 1 "GNDPWR" H 7004 1696 50  0000 C CNN
-F 2 "" H 7000 1800 50  0001 C CNN
-F 3 "" H 7000 1800 50  0001 C CNN
-	1    7000 1850
-	1    0    0    -1
-$EndComp
-$Comp
 L Device:R_Small R16
 U 1 1 5CD8E6F8
@@
 F 3 "~" H 5800 1550 50  0001 C CNN
 	1    5800 1550
-	1    0    0    -1
-$EndComp
-$Comp
-L power:GNDPWR #PWR0120
-U 1 1 5CDA966A
-P 4900 1850
-F 0 "#PWR0120" H 4900 1650 50  0001 C CNN
-F 1 "GNDPWR" H 4904 1696 50  0000 C CNN
-F 2 "" H 4900 1800 50  0001 C CNN
-F 3 "" H 4900 1800 50  0001 C CNN
-	1    4900 1850
 	1    0    0    -1
 $EndComp
@@
 	-1   0    0    1
 $EndComp
-$Comp
-L power:GNDPWR #PWR0121
-U 1 1 5CDE5124
-P 6650 1850
-F 0 "#PWR0121" H 6650 1650 50  0001 C CNN
-F 1 "GNDPWR" H 6654 1696 50  0000 C CNN
-F 2 "" H 6650 1800 50  0001 C CNN
-F 3 "" H 6650 1800 50  0001 C CNN
-	1    6650 1850
-	1    0    0    -1
-$EndComp
 Wire Wire Line
 	6000 2100 6000 2050
@@
 	1    0    0    -1
 $EndComp
-$Comp
-L power:GNDPWR #PWR0122
-U 1 1 5CE10BAA
-P 6000 2800
-F 0 "#PWR0122" H 6000 2600 50  0001 C CNN
-F 1 "GNDPWR" H 6004 2646 50  0000 C CNN
-F 2 "" H 6000 2750 50  0001 C CNN
-F 3 "" H 6000 2750 50  0001 C CNN
-	1    6000 2800
-	1    0    0    -1
-$EndComp
 Text GLabel 1650 2550 0    50   Input ~ 0
 VP
@@
 $EndComp
 $Comp
-L power:GNDPWR #PWR0123
-U 1 1 5CE1B512
-P 5150 1850
-F 0 "#PWR0123" H 5150 1650 50  0001 C CNN
-F 1 "GNDPWR" H 5154 1696 50  0000 C CNN
-F 2 "" H 5150 1800 50  0001 C CNN
-F 3 "" H 5150 1800 50  0001 C CNN
-	1    5150 1850
-	1    0    0    -1
-$EndComp
-$Comp
 L Device:C_Small C23
 U 1 1 5CE24551
@@
 $EndComp
 $Comp
-L power:GNDPWR #PWR0124
-U 1 1 5CE24557
-P 6550 1300
-F 0 "#PWR0124" H 6550 1100 50  0001 C CNN
-F 1 "GNDPWR" H 6750 1250 50  0000 C CNN
-F 2 "" H 6550 1250 50  0001 C CNN
-F 3 "" H 6550 1250 50  0001 C CNN
-	1    6550 1300
-	1    0    0    -1
-$EndComp
-$Comp
 L Device:C_Small C25
 U 1 1 5CE366FA
@@
 F 3 "~" H 7300 1750 50  0001 C CNN
 	1    7300 1750
-	1    0    0    -1
-$EndComp
-$Comp
-L power:GNDPWR #PWR0125
-U 1 1 5CE36700
-P 7300 1850
-F 0 "#PWR0125" H 7300 1650 50  0001 C CNN
-F 1 "GNDPWR" H 7304 1696 50  0000 C CNN
-F 2 "" H 7300 1800 50  0001 C CNN
-F 3 "" H 7300 1800 50  0001 C CNN
-	1    7300 1850
 	1    0    0    -1
 $EndComp
@@
 	1    0    0    -1
 $EndComp
+$Comp
+L power:GND #PWR?
+U 1 1 5CEBEE53
+P 6000 2800
+F 0 "#PWR?" H 6000 2550 50  0001 C CNN
+F 1 "GND" H 6005 2627 50  0000 C CNN
+F 2 "" H 6000 2800 50  0001 C CNN
+F 3 "" H 6000 2800 50  0001 C CNN
+	1    6000 2800
+	1    0    0    -1
+$EndComp
+$Comp
+L power:GND #PWR?
+U 1 1 5CEBF779
+P 7300 1850
+F 0 "#PWR?" H 7300 1600 50  0001 C CNN
+F 1 "GND" H 7305 1677 50  0000 C CNN
+F 2 "" H 7300 1850 50  0001 C CNN
+F 3 "" H 7300 1850 50  0001 C CNN
+	1    7300 1850
+	1    0    0    -1
+$EndComp
+$Comp
+L power:GND #PWR?
+U 1 1 5CEC0041
+P 7000 1850
+F 0 "#PWR?" H 7000 1600 50  0001 C CNN
+F 1 "GND" H 7005 1677 50  0000 C CNN
+F 2 "" H 7000 1850 50  0001 C CNN
+F 3 "" H 7000 1850 50  0001 C CNN
+	1    7000 1850
+	1    0    0    -1
+$EndComp
+$Comp
+L power:GND #PWR?
+U 1 1 5CEC032A
+P 6650 1850
+F 0 "#PWR?" H 6650 1600 50  0001 C CNN
+F 1 "GND" H 6655 1677 50  0000 C CNN
+F 2 "" H 6650 1850 50  0001 C CNN
+F 3 "" H 6650 1850 50  0001 C CNN
+	1    6650 1850
+	1    0    0    -1
+$EndComp
+$Comp
+L power:GND #PWR?
+U 1 1 5CEC71E6
+P 6550 1300
+F 0 "#PWR?" H 6550 1050 50  0001 C CNN
+F 1 "GND" H 6555 1127 50  0000 C CNN
+F 2 "" H 6550 1300 50  0001 C CNN
+F 3 "" H 6550 1300 50  0001 C CNN
+	1    6550 1300
+	1    0    0    -1
+$EndComp
+$Comp
+L power:GND #PWR?
+U 1 1 5CECE198
+P 6250 1300
+F 0 "#PWR?" H 6250 1050 50  0001 C CNN
+F 1 "GND" H 6255 1127 50  0000 C CNN
+F 2 "" H 6250 1300 50  0001 C CNN
+F 3 "" H 6250 1300 50  0001 C CNN
+	1    6250 1300
+	1    0    0    -1
+$EndComp
+$Comp
+L power:GND #PWR?
+U 1 1 5CED510C
+P 4900 1850
+F 0 "#PWR?" H 4900 1600 50  0001 C CNN
+F 1 "GND" H 4905 1677 50  0000 C CNN
+F 2 "" H 4900 1850 50  0001 C CNN
+F 3 "" H 4900 1850 50  0001 C CNN
+	1    4900 1850
+	1    0    0    -1
+$EndComp
+$Comp
+L power:GND #PWR?
+U 1 1 5CEDC0E0
+P 5150 1850
+F 0 "#PWR?" H 5150 1600 50  0001 C CNN
+F 1 "GND" H 5155 1677 50  0000 C CNN
+F 2 "" H 5150 1850 50  0001 C CNN
+F 3 "" H 5150 1850 50  0001 C CNN
+	1    5150 1850
+	1    0    0    -1
+$EndComp

Commit message: finalized board, silkscreen needs some work
Parts:
- removed C27, C4: 100n, Capacitor_SMD:C_0603_1608Metric, symbol Device:C_Small
Changed lines of the file:
@@
 $EndComp
-$Comp
-L power:GND #PWR0139
-U 1 1 5CE919A0
-P 6650 5800
-F 0 "#PWR0139" H 6650 5550 50  0001 C CNN
-F 1 "GND" H 6655 5627 50  0000 C CNN
-F 2 "" H 6650 5800 50  0001 C CNN
-F 3 "" H 6650 5800 50  0001 C CNN
-	1    6650 5800
-	1    0    0    -1
-$EndComp
-$Comp
-L Device:C_Small C27
-U 1 1 5CE9199A
-P 6650 5700
-F 0 "C27" H 6742 5746 50  0000 L CNN
-F 1 "100n" H 6742 5655 50  0000 L CNN
-F 2 "Capacitor_SMD:C_0603_1608Metric" H 6650 5700 50  0001 C CNN
-F 3 "~" H 6650 5700 50  0001 C CNN
-	1    6650 5700
-	1    0    0    -1
-$EndComp
-Text GLabel 6650 5600 1    50   Input ~ 0
-VIO
 $Comp
 L power:GND #PWR0137
@@
 	1    0    0    -1
 $EndComp
-$Comp
-L power:GND #PWR0116
-U 1 1 5CD01E0F
-P 6300 5800
-F 0 "#PWR0116" H 6300 5550 50  0001 C CNN
-F 1 "GND" H 6305 5627 50  0000 C CNN
-F 2 "" H 6300 5800 50  0001 C CNN
-F 3 "" H 6300 5800 50  0001 C CNN
-	1    6300 5800
-	1    0    0    -1
-$EndComp
-$Comp
-L Device:C_Small C4
-U 1 1 5CD01E09
-P 6300 5700
-F 0 "C4" H 6392 5746 50  0000 L CNN
-F 1 "100n" H 6392 5655 50  0000 L CNN
-F 2 "Capacitor_SMD:C_0603_1608Metric" H 6300 5700 50  0001 C CNN
-F 3 "~" H 6300 5700 50  0001 C CNN
-	1    6300 5700
-	1    0    0    -1
-$EndComp
-Text GLabel 6300 5600 1    50   Input ~ 0
-VIO
 $Comp
 L power:GND #PWR0114
@@
 $EndComp
 $Comp
-L power:GND #PWR?
+L power:GND #PWR0118
 U 1 1 5CEBEE53
 P 6000 2800
-F 0 "#PWR?" H 6000 2550 50  0001 C CNN
+F 0 "#PWR0118" H 6000 2550 50  0001 C CNN
 F 1 "GND" H 6005 2627 50  0000 C CNN
 F 2 "" H 6000 2800 50  0001 C CNN
@@
 $EndComp
 $Comp
-L power:GND #PWR?
+L power:GND #PWR0119
 U 1 1 5CEBF779
 P 7300 1850
-F 0 "#PWR?" H 7300 1600 50  0001 C CNN
+F 0 "#PWR0119" H 7300 1600 50  0001 C CNN
 F 1 "GND" H 7305 1677 50  0000 C CNN
 F 2 "" H 7300 1850 50  0001 C CNN
@@
 $EndComp
 $Comp
-L power:GND #PWR?
+L power:GND #PWR0120
 U 1 1 5CEC0041
 P 7000 1850
-F 0 "#PWR?" H 7000 1600 50  0001 C CNN
+F 0 "#PWR0120" H 7000 1600 50  0001 C CNN
 F 1 "GND" H 7005 1677 50  0000 C CNN
 F 2 "" H 7000 1850 50  0001 C CNN
@@
 $EndComp
 $Comp
-L power:GND #PWR?
+L power:GND #PWR0121
 U 1 1 5CEC032A
 P 6650 1850
-F 0 "#PWR?" H 6650 1600 50  0001 C CNN
+F 0 "#PWR0121" H 6650 1600 50  0001 C CNN
 F 1 "GND" H 6655 1677 50  0000 C CNN
 F 2 "" H 6650 1850 50  0001 C CNN
@@
 $EndComp
 $Comp
-L power:GND #PWR?
+L power:GND #PWR0122
 U 1 1 5CEC71E6
 P 6550 1300
-F 0 "#PWR?" H 6550 1050 50  0001 C CNN
+F 0 "#PWR0122" H 6550 1050 50  0001 C CNN
 F 1 "GND" H 6555 1127 50  0000 C CNN
 F 2 "" H 6550 1300 50  0001 C CNN
@@
 $EndComp
 $Comp
-L power:GND #PWR?
+L power:GND #PWR0123
 U 1 1 5CECE198
 P 6250 1300
-F 0 "#PWR?" H 6250 1050 50  0001 C CNN
+F 0 "#PWR0123" H 6250 1050 50  0001 C CNN
 F 1 "GND" H 6255 1127 50  0000 C CNN
 F 2 "" H 6250 1300 50  0001 C CNN
@@
 $EndComp
 $Comp
-L power:GND #PWR?
+L power:GND #PWR0124
 U 1 1 5CED510C
 P 4900 1850
-F 0 "#PWR?" H 4900 1600 50  0001 C CNN
+F 0 "#PWR0124" H 4900 1600 50  0001 C CNN
 F 1 "GND" H 4905 1677 50  0000 C CNN
 F 2 "" H 4900 1850 50  0001 C CNN
@@
 $EndComp
 $Comp
-L power:GND #PWR?
+L power:GND #PWR0125
 U 1 1 5CEDC0E0
 P 5150 1850
-F 0 "#PWR?" H 5150 1600 50  0001 C CNN
+F 0 "#PWR0125" H 5150 1600 50  0001 C CNN
 F 1 "GND" H 5155 1677 50  0000 C CNN
 F 2 "" H 5150 1850 50  0001 C CNN
