File: PAC5523/PAC5523.sch (KiCad schematic (older format))
At the start: 68 parts, among them J1 W, J2 U, J3 V, Q1 AON6276, U1 PAC5523, U10 PA1137NL, U4 Oscillator_3225

Commit message: updated files
Other:
- note removed: "Gate Pulldowns!\n"
Changed lines of the file:
@@
 EESchema Schematic File Version 4
 LIBS:PAC5523-cache
-EELAYER 29 0
+EELAYER 26 0
 EELAYER END
 $Descr A4 11693 8268
@@
 Text Notes 7050 1450 0    50   ~ 0
 Für Design < 20V brücke vorsehen\n
-Text Notes 10250 850  0    50   ~ 0
-Gate Pulldowns!\n
 $EndSCHEMATC
