File: PAC5523/PAC5523.kicad_pcb (KiCad board)
At the start: 4 copper layers, 60 x 44 mm, 128 parts, among them J1 W, J10 NTC, J11 LED, J2 U, J3 V, J4 GND, J5 VIN, J6 UART, J7 ENCODER, J8 HALL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

Commit message: added notes
Parts:
- C32: value TBD -> 1n
- R1, R8, R9: value TBD -> 5.1
- R10, R11, R12, R13, R15, R2, R3: value 22 -> 10
- R14: value TBD -> 0.3
- R16: value TBD -> 0
- R36: value TBD -> 220
- R38: value 9k6 -> 9k1
Changed lines of the file:
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@@
     (1 In1.Cu mixed)
     (2 In2.Cu power)
-    (31 B.Cu power hide)
+    (31 B.Cu power)
     (33 F.Adhes user)
     (34 B.Paste user)
@@
   )
   (setup
-    (last_trace_width 0.154)
+    (last_trace_width 0.2)
     (user_trace_width 0.154)
     (user_trace_width 0.2)
@@
     (pcbplotparams
       (layerselection 0x010fc_ffffffff)
-      (usegerberextensions false)
+      (usegerberextensions true)
       (usegerberattributes false)
       (usegerberadvancedattributes false)
       (creategerberjobfile false)
-      (excludeedgelayer true)
+      (excludeedgelayer false)
       (linewidth 0.100000)
       (plotframeref false)
@@
       (outputformat 1)
       (mirror false)
-      (drillshape 1)
+      (drillshape 0)
       (scaleselection 1)
-      (outputdirectory ""))
+      (outputdirectory "gerber/"))
   )
   (net 0 "")
@@
       (effects (font (size 0.4 0.4) (thickness 0.1)))
     )
-    (fp_text value 9k6 (at 0 1.43 90) (layer F.Fab)
+    (fp_text value 9k1 (at 0 1.43 90) (layer F.Fab)
       (effects (font (size 1 1) (thickness 0.15)))
     )
@@
       (effects (font (size 0.4 0.4) (thickness 0.1)))
     )
-    (fp_text value TBD (at 0 1.43) (layer F.Fab)
+    (fp_text value 5.1 (at 0 1.43) (layer F.Fab)
       (effects (font (size 1 1) (thickness 0.15)))
     )
@@
       (effects (font (size 0.4 0.4) (thickness 0.1)))
     )
-    (fp_text value TBD (at 0 1.65 180) (layer F.Fab)
+    (fp_text value 0.3 (at 0 1.65 180) (layer F.Fab)
       (effects (font (size 1 1) (thickness 0.15)))
     )
@@
       (effects (font (size 0.4 0.4) (thickness 0.1)))
     )
-    (fp_text value 22 (at 0 1.65 270) (layer F.Fab)
+    (fp_text value 10 (at 0 1.65 270) (layer F.Fab)
       (effects (font (size 1 1) (thickness 0.15)))
     )
@@
       (effects (font (size 0.4 0.4) (thickness 0.1)))
     )
-    (fp_text value 22 (at 0 1.65 180) (layer F.Fab)
+    (fp_text value 10 (at 0 1.65 180) (layer F.Fab)
       (effects (font (size 1 1) (thickness 0.15)))
     )
@@
       (effects (font (size 0.4 0.4) (thickness 0.1)))
     )
-    (fp_text value 22 (at 0 1.65 180) (layer F.Fab)
+    (fp_text value 10 (at 0 1.65 180) (layer F.Fab)
       (effects (font (size 1 1) (thickness 0.15)))
     )
@@
       (effects (font (size 0.4 0.4) (thickness 0.1)))
     )
-    (fp_text value 22 (at 0 1.65 180) (layer F.Fab)
+    (fp_text value 10 (at 0 1.65 180) (layer F.Fab)
       (effects (font (size 1 1) (thickness 0.15)))
     )
@@
       (effects (font (size 0.4 0.4) (thickness 0.1)))
     )
-    (fp_text value 22 (at 0 1.65 180) (layer F.Fab)
+    (fp_text value 10 (at 0 1.65 180) (layer F.Fab)
       (effects (font (size 1 1) (thickness 0.15)))
     )
@@
       (effects (font (size 0.4 0.4) (thickness 0.1)))
     )
-    (fp_text value TBD (at 0 1.43 270) (layer F.Fab)
+    (fp_text value 5.1 (at 0 1.43 270) (layer F.Fab)
       (effects (font (size 1 1) (thickness 0.15)))
     )
@@
       (effects (font (size 0.4 0.4) (thickness 0.1)))
     )
-    (fp_text value TBD (at 0 1.43 90) (layer F.Fab)
+    (fp_text value 5.1 (at 0 1.43 90) (layer F.Fab)
       (effects (font (size 1 1) (thickness 0.15)))
     )
@@
       (effects (font (size 0.4 0.4) (thickness 0.1)))
     )
-    (fp_text value 22 (at 0 1.65) (layer F.Fab)
+    (fp_text value 10 (at 0 1.65) (layer F.Fab)
       (effects (font (size 1 1) (thickness 0.15)))
     )
@@
       (effects (font (size 0.4 0.4) (thickness 0.1)))
     )
-    (fp_text value 22 (at 0 1.65) (layer F.Fab)
+    (fp_text value 10 (at 0 1.65) (layer F.Fab)
       (effects (font (size 1 1) (thickness 0.15)))
     )
@@
       (effects (font (size 0.4 0.4) (thickness 0.1)))
     )
-    (fp_text value TBD (at 0 1.43) (layer F.Fab)
+    (fp_text value 220 (at 0 1.43) (layer F.Fab)
       (effects (font (size 1 1) (thickness 0.15)))
     )
@@
       (effects (font (size 0.4 0.4) (thickness 0.1)))
     )
-    (fp_text value TBD (at 0 1.43 180) (layer F.Fab)
+    (fp_text value 0 (at 0 1.43 180) (layer F.Fab)
       (effects (font (size 1 1) (thickness 0.15)))
     )
@@
       (effects (font (size 0.4 0.4) (thickness 0.1)))
     )
-    (fp_text value TBD (at 0 1.43 180) (layer F.Fab)
+    (fp_text value 1n (at 0 1.43 180) (layer F.Fab)
       (effects (font (size 1 1) (thickness 0.15)))
     )
@@
   (gr_line (start 80 67) (end 20 67) (layer Edge.Cuts) (width 0.05))
   (gr_line (start 80 23) (end 80 67) (layer Edge.Cuts) (width 0.05))
-  (via (at 35.61 53.23) (size 0.6) (drill 0.3) (layers F.Cu B.Cu) (net 43))
-  (via (at 37.46 61.58) (size 0.6) (drill 0.3) (layers F.Cu B.Cu) (net 43))
   (segment (start 62.32 33.82) (end 62.32 33.6875) (width 0.154) (layer F.Cu) (net 1))
   (segment (start 63.3 35.35) (end 63.3 34.8) (width 0.154) (layer F.Cu) (net 1))
@@
   (segment (start 47.5875 62.0125) (end 47.5875 60.1) (width 0.8) (layer F.Cu) (net 35))
   (segment (start 46.5 63.1) (end 47.5875 62.0125) (width 0.8) (layer F.Cu) (net 35))
-  (segment (start 38 44.0125) (end 37.2875 43.3) (width 0.4) (layer F.Cu) (net 91))
-  (segment (start 38 44.95) (end 38 44.0125) (width 0.4) (layer F.Cu) (net 91))
   (segment (start 73.405 56.65) (end 73.7875 56.65) (width 0.4) (layer F.Cu) (net 36))
   (segment (start 33.2125 28.5) (end 33.8125 29.1) (width 0.4) (layer F.Cu) (net 36))
@@
   (segment (start 61.047782 39.34599) (end 60.094447 40.299325) (width 0.2) (layer F.Cu) (net 42))
   (segment (start 60.094447 40.299325) (end 60.094447 40.604909) (width 0.2) (layer F.Cu) (net 42))
+  (via (at 35.61 53.23) (size 0.6) (drill 0.3) (layers F.Cu B.Cu) (net 43))
+  (via (at 37.46 61.58) (size 0.6) (drill 0.3) (layers F.Cu B.Cu) (net 43))
   (segment (start 35.7 50.355) (end 35.7 49.695) (width 0.8) (layer F.Cu) (net 43))
   (segment (start 34.08 51.975) (end 35.7 50.355) (width 0.8) (layer F.Cu) (net 43))
@@
   (segment (start 37.416022 25.083978) (end 32.35 30.15) (width 0.154) (layer In1.Cu) (net 63))
   (segment (start 67.450749 39.598232) (end 67.450749 33.570435) (width 0.154) (layer In1.Cu) (net 63))
-  (segment (start 67.805 58.38) (end 67.925 58.5) (width 0.2) (layer F.Cu) (net 92))
-  (segment (start 67.805 56.65) (end 67.805 58.38) (width 0.2) (layer F.Cu) (net 92))
-  (segment (start 39.7125 47.3) (end 39.7 47.2875) (width 0.2) (layer F.Cu) (net 93))
-  (segment (start 41.3 47.3) (end 39.7125 47.3) (width 0.2) (layer F.Cu) (net 93))
-  (segment (start 38.4375 47.2875) (end 38 46.85) (width 0.2) (layer F.Cu) (net 93))
-  (segment (start 39.7 47.2875) (end 38.4375 47.2875) (width 0.2) (layer F.Cu) (net 93))
   (segment (start 68.164408 36.5) (end 68.306009 36.358399) (width 0.154) (layer F.Cu) (net 64))
   (segment (start 68.306009 36.358399) (end 68.306009 35.933599) (width 0.154) (layer F.Cu) (net 64))
@@
   (segment (start 59.7125 58.2) (end 59.575 58.0625) (width 0.154) (layer F.Cu) (net 88))
   (segment (start 59.7125 59.5) (end 59.7125 58.2) (width 0.154) (layer F.Cu) (net 88))
+  (segment (start 38 44.0125) (end 37.2875 43.3) (width 0.4) (layer F.Cu) (net 91))
+  (segment (start 38 44.95) (end 38 44.0125) (width 0.4) (layer F.Cu) (net 91))
+  (segment (start 67.805 58.38) (end 67.925 58.5) (width 0.2) (layer F.Cu) (net 92))
+  (segment (start 67.805 56.65) (end 67.805 58.38) (width 0.2) (layer F.Cu) (net 92))
+  (segment (start 39.7125 47.3) (end 39.7 47.2875) (width 0.2) (layer F.Cu) (net 93))
+  (segment (start 41.3 47.3) (end 39.7125 47.3) (width 0.2) (layer F.Cu) (net 93))
+  (segment (start 38.4375 47.2875) (end 38 46.85) (width 0.2) (layer F.Cu) (net 93))
+  (segment (start 39.7 47.2875) (end 38.4375 47.2875) (width 0.2) (layer F.Cu) (net 93))
   (zone (net 10) (net_name GND) (layer B.Cu) (hatch edge 0.508)
     (priority 1)
