File: STM32G431/PAC5523.kicad_pcb (KiCad board)
At the start: 4 copper layers, 60 x 44 mm, 128 parts, among them J1 W, J10 NTC, J11 LED, J2 U, J3 V, J4 GND, J5 VIN, J6 UART, J7 ENCODER, J8 HALL, J9 AIN, P1 TC2030-CTX-Tag-Connect, Q1 AON6276, Q2 Q_NMOS_GSD, U1 PAC5523, U10 PA1137NL, U11 USBLC6-4, U2 MAX3051, U3 ACT4088, U4 Oscillator_3225, U5 RS485, U6 ENCODER A, U7 ENCODER B, U8 USBLC6-4, U9 USBLC6-4

Commit message: updated files
Parts:
- removed D16, D18, D19: SS310, Diode_SMD:D_SOD-123F
- removed J7: ENCODER, Connector_Molex:Molex_PicoBlade_53261-0671_1x06-1MP_P1.25mm_Horizontal
- removed Q1: AON6276, Package_SON:VSONP-8-1EP_5x6_P1.27mm
- removed R18, R22: 120, Resistor_SMD:R_0603_1608Metric
- added C38: 10u, Capacitor_SMD:C_1206_3216Metric, F.Cu at (70.3, -3.14)
- added C43: 100n 100V, Capacitor_SMD:C_0603_1608Metric, F.Cu at (78.1, -7.03)
- added C44: 100p, Capacitor_SMD:C_0603_1608Metric, F.Cu at (57.2, 11.7)
- added C45: 100p, Capacitor_SMD:C_0603_1608Metric, F.Cu at (75.1, -3.53)
- added C46: 100n 100V, Capacitor_SMD:C_0603_1608Metric, F.Cu at (59.5, 9.21)
- added C47: 4u7, Capacitor_SMD:C_0603_1608Metric, F.Cu at (38.5, 36.4)
- added C48: 4u7, Capacitor_SMD:C_0603_1608Metric, F.Cu at (38.5, 38.9)
- added C49: 4u7, Capacitor_SMD:C_0603_1608Metric, F.Cu at (56.9, 29.9)
- added FB1: FERRET, Inductor_SMD:L_0805_2012Metric, F.Cu at (78.3, -9.76)
- added L2: 100u 1A, Inductor_SMD:L_Taiyo-Yuden_MD-4040, F.Cu at (42.5, -5.36)
- added R40: 1.5k, Resistor_SMD:R_0603_1608Metric, F.Cu at (69.5, -0.24)
- added R41: 1.5k, Resistor_SMD:R_0603_1608Metric, F.Cu at (73.5, 2.27)
- added R42: 1.5k, Resistor_SMD:R_0603_1608Metric, F.Cu at (73.2, 9.80)
- added U12: AMS1117-3.3, Package_TO_SOT_SMD:SOT-223-3_TabPin2, F.Cu at (54.3, -7.11)
- added Y1: 8Mhz, Crystal:Crystal_SMD_3225-4Pin_3.2x2.5mm, F.Cu at (60.1, 5.73)
- C1, C11, C12: value 1uF -> 22uF
- C13, C14, C15, C16, C2, C3: value TBD -> DNP
- C17: value 100p -> 4u7
- C18: value 100p -> 100n
- C20: value 10u -> 33n; footprint Capacitor_SMD:C_1206_3216Metric -> Capacitor_SMD:C_0603_1608Metric
- C21: value 100n -> 100n 100V
- C22: value 4u7 -> 100n 100V
- C23: value 100n -> 10u; footprint Capacitor_SMD:C_0603_1608Metric -> Capacitor_SMD:C_1206_3216Metric
- C32: value 1n -> 100n
- C33: value 10u -> 100n; footprint Capacitor_SMD:C_1206_3216Metric -> Capacitor_SMD:C_0603_1608Metric
- C4, C5: value 100n -> 18p
- C41: value 18p -> 10u; footprint Capacitor_SMD:C_0603_1608Metric -> Capacitor_SMD:C_1206_3216Metric
- C6: value 4u7 -> 100n
- C7: value 4u7 -> 100u 100V; footprint Capacitor_SMD:C_0603_1608Metric -> Capacitor_THT:CP_Radial_D8.0mm_P3.80mm
- D1, D11, D12, D14, D15, D3, D4, D8, D9: value SS310 -> SM4007PL
- D10, D13, D2, D5, D6, D7: value SS310 -> B5819W; footprint Diode_SMD:D_SOD-123F -> Diode_SMD:D_SOD-123
- J9: value AIN -> AIN/PWM; footprint Connector_Molex:Molex_PicoBlade_53261-0371_1x03-1MP_P1.25mm_Horizontal -> Connector_Molex:Molex_PicoBlade_53261-0471_1x04-1MP_P1.25mm_Horizontal
- R1, R8: value 5.1 -> 22k
- R10, R11, R12, R13, R2, R3: value 10 -> 2
- R14: value 0.3 -> 22k; footprint Resistor_SMD:R_0805_2012Metric -> Resistor_SMD:R_0603_1608Metric
- R15: value 10 -> 2.2k; footprint Resistor_SMD:R_0805_2012Metric -> Resistor_SMD:R_0603_1608Metric
- R16: value 0 -> 22k
- R36: value 220 -> 2.2k
- R7: value 51 -> 2.7k
- R9: value 5.1 -> 2.2k
- U1: value PAC5523 -> STM32G431CBUx
- U10: value PA1137NL -> MIC4605; footprint otter:PA1137NL -> Package_SO:SOIC-8_3.9x4.9mm_P1.27mm
- U4: value Oscillator_3225 -> XL7015; footprint otter:Oscillator_3225 -> Package_TO_SOT_SMD:TO-252-5_TabPin3
- U6: value ENCODER A -> MIC4605
- U7: value ENCODER B -> MIC4605
- moved D13 102.0 mm to (101.5, -6.21), turned to 0 degrees
- moved D15 87.4 mm to (78.9, -16.8), turned to 0 degrees
- moved C20 83.9 mm to (79.2, -4.52), turned to 0 degrees
- moved D14 82.0 mm to (73.5, -16.8)
- moved J9 77.1 mm to (92.2, -7.01)
- moved R26 73.0 mm to (106.4, -9.98)
- moved C25 69.6 mm to (69.5, 2.27), turned to 0 degrees
- moved R16 69.2 mm to (72.8, 7.29), turned to 0 degrees
- moved D2 65.5 mm to (101.5, -9.56), turned to 0 degrees
- moved D7 64.8 mm to (105.8, -2.86), turned to 0 degrees
- moved R14 64.7 mm to (77.5, 1.49), turned to 0 degrees
- moved C33 63.0 mm to (64.8, 4.76), turned to 0 degrees
- moved D10 62.7 mm to (100.0, -1.71), turned to 0 degrees
- moved R1 62.3 mm to (73.5, -0.24)
- moved D5 58.1 mm to (94.3, -1.71), turned to 0 degrees
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Connections:
- C1 pad 1: DRB5 -> Net-(C1-Pad1)
- C1 pad 2: DRS5 -> U
- C11 pad 1: DRB4 -> Net-(C11-Pad1)
- C11 pad 2: DRS4 -> V
- C12 pad 1: DRB3 -> Net-(C12-Pad1)
- C12 pad 2: DRS3 -> W
- C17 pad 1: IUH -> VDDA
- C17 pad 2: IUL -> GND
- C18 pad 1: IVH -> VDDA
- C18 pad 2: IVL -> GND
- C20 pad 1: Net-(C20-Pad1) -> +12V
- C20 pad 2: GND -> Net-(C20-Pad2)
- C21 pad 1: Net-(C20-Pad1) -> VIN
- C22 pad 1: VHM -> +12V
- C23 pad 1: VHM -> +12V
- C24 pad 1: +5V -> +3V3
- C25 pad 1: VP -> +12V
- C26 pad 1: +5V -> +3V3
- C28 pad 1: +5V -> +3V3
- C32 pad 1: Net-(C20-Pad1) -> +12V
- C32 pad 2: Net-(C32-Pad2) -> GND
- C33 pad 1: VP -> +12V
- C34 pad 1: +5V -> +3V3
- C4 pad 1: VIO -> Net-(C4-Pad1)
- C41 pad 1: CLK -> +12V
- C5 pad 1: VIO -> Net-(C5-Pad1)
- C6 pad 1: VCC18 -> NRST
- C7 pad 1: VCORE -> VIN
- C8 pad 1: VIO -> +3V3
- C9 pad 1: 3V3 -> +3V3
- D1 pad 1: DRS5 -> Net-(D1-Pad1)
- D10 pad 1: DRB3 -> +3V3
- D10 pad 2: VP -> UW
- D11 pad 1: DRH3 -> Net-(D11-Pad1)
- D12 pad 1: DRL0 -> Net-(D12-Pad1)
- D13 pad 1: Net-(C20-Pad1) -> GPIO_BEMF
- D13 pad 2: VIN -> Net-(D13-Pad2)
- D14 pad 1: VP -> Net-(C35-Pad2)
- D14 pad 2: Net-(D14-Pad2) -> GND
- D15 pad 1: VHM -> Net-(C40-Pad1)
- D15 pad 2: VP -> NTC_EXT
- D2 pad 1: DRB5 -> +3V3
- D2 pad 2: VP -> UU
- D3 pad 1: DRH5 -> Net-(D3-Pad1)
- D4 pad 1: DRL2 -> Net-(D4-Pad1)
- D5 pad 1: DRS4 -> GPIO_BEMF
- D5 pad 2: GND -> Net-(D5-Pad2)
- D6 pad 1: DRS3 -> +3V3
- D6 pad 2: GND -> UV
- D7 pad 1: DRB4 -> GPIO_BEMF
- D7 pad 2: VP -> Net-(D7-Pad2)
- D8 pad 1: DRH4 -> Net-(D8-Pad1)
- D9 pad 1: DRL1 -> Net-(D9-Pad1)
- J1 pad 3: IWH -> Net-(J1-Pad3)
- J2 pad 3: IUH -> Net-(J2-Pad3)
- J3 pad 3: IVH -> Net-(J3-Pad3)
- J9 pad 2: Net-(J9-Pad2) -> PWM
- J9 pad 3: GND -> Net-(J9-Pad3)
- P1 pad 4: SWDCL -> SWCLK
- R1 pad 1: U -> Net-(C20-Pad2)
- R1 pad 2: DRS5 -> +12V
- R10 pad 2: DRH4 -> Net-(D8-Pad1)
- R11 pad 2: DRL1 -> Net-(D9-Pad1)
- R12 pad 2: DRH3 -> Net-(D11-Pad1)
- R13 pad 2: DRL0 -> Net-(D12-Pad1)
- R14 pad 1: CSM -> IVH
- R14 pad 2: GND -> +3V3
- R15 pad 1: DRM -> GND
- R15 pad 2: Net-(Q1-Pad2) -> IVH
- R16 pad 1: VHM -> IWH
- R16 pad 2: Net-(C20-Pad1) -> +3V3
- R2 pad 2: DRH5 -> Net-(D3-Pad1)
- R24 pad 1: UU -> Net-(D5-Pad2)
- R24 pad 2: GND -> UU
- R26 pad 1: UV -> Net-(D7-Pad2)
- R26 pad 2: GND -> UV
- R3 pad 2: DRL2 -> Net-(D4-Pad1)
- R30 pad 1: W -> UW
- R30 pad 2: UW -> W
- R31 pad 1: UW -> Net-(D13-Pad2)
- R31 pad 2: GND -> UW
- R36 pad 1: Net-(C32-Pad2) -> GND
- R36 pad 2: Net-(C20-Pad1) -> IWH
- R4 pad 2: CANTX -> UART_RX
- R45 pad 2: Net-(J9-Pad2) -> Net-(J9-Pad3)
- R46 pad 2: Net-(J9-Pad2) -> Net-(J9-Pad3)
- R5 pad 2: CANRX -> UART_TX
- R7 pad 1: VSYS -> GND
- R7 pad 2: Net-(R7-Pad2) -> Net-(C20-Pad2)
- R8 pad 1: V -> IUH
- R8 pad 2: DRS4 -> +3V3
- R9 pad 1: W -> GND
- R9 pad 2: DRS3 -> IUH
- U1 pad 1: ENC_B -> +3V3
- U1 pad 10: IUH -> Net-(U1-Pad10)
- U1 pad 11: Ain -> IUL
- U1 pad 13: UV -> IVL
- U1 pad 14: UW -> Net-(U1-Pad14)
- U1 pad 15: VSYS -> IVH
- U1 pad 16: Net-(R7-Pad2) -> UV
- U1 pad 17: CSM -> IWH
- U1 pad 18: VP -> Net-(U1-Pad18)
- U1 pad 19: VHM -> IWL
- U1 pad 2: ENC_A -> UL
- U1 pad 20: DRM -> VDDA
- U1 pad 21: DRL0 -> VDDA
- U1 pad 22: DRL1 -> Net-(U1-Pad22)
- U1 pad 23: DRL2 -> +3V3
- U1 pad 24: DRS3 -> UW
- U1 pad 25: DRH3 -> Ain
- U1 pad 26: DRB3 -> Net-(U1-Pad26)
- U1 pad 27: DRS4 -> NTC_IO
- U1 pad 28: DRH4 -> WL
- U1 pad 29: DRB4 -> SK6812
- U1 pad 3: SWDCL -> Net-(U1-Pad3)
- U1 pad 30: DRS5 -> UH
- U1 pad 31: DRH5 -> VH
- U1 pad 32: DRB5 -> WH
- U1 pad 33: SK6812 -> CANRX
- U1 pad 34: CANRX -> VL
- U1 pad 35: CANTX -> +3V3
- U1 pad 36: HALL1 -> SWDIO
- U1 pad 37: HALL2 -> SWCLK
- U1 pad 38: HALL3 -> PWM
- U1 pad 39: CLK -> Net-(U1-Pad39)
- U1 pad 4: 3V3 -> Net-(U1-Pad4)
- U1 pad 41: VCC18 -> UART_TX
- U1 pad 42: VCORE -> UART_RX
- U1 pad 43: GND -> GPIO_BEMF
- U1 pad 44: VIO -> HALL1
- U1 pad 45: NTC_IO -> HALL2
- U1 pad 46: SWDIO -> HALL3
- U1 pad 47: Vin_mon -> CANTX
- U1 pad 48: Net-(U1-Pad48) -> +3V3
- U1 pad 5: IWL -> Net-(C4-Pad1)
- U1 pad 6: IWH -> Net-(C5-Pad1)
- U1 pad 7: IVL -> NRST
- U1 pad 8: IVH -> Vin_mon
- U1 pad 9: IUL -> IUH
- U10 pad 1: Net-(U10-Pad1) -> +12V
- U10 pad 2: Net-(U10-Pad2) -> Net-(C12-Pad1)
- U10 pad 3: Net-(D16-Pad2) -> Net-(D11-Pad1)
- U10 pad 4: Net-(C20-Pad1) -> W
- U10 pad 5: (no net) -> WH
- U10 pad 6: (no net) -> WL
- U10 pad 7: Net-(D14-Pad2) -> GND
- U10 pad 8: Net-(D14-Pad2) -> Net-(D12-Pad1)
- U11 pad 1: CANRX -> Net-(U11-Pad1)
- U11 pad 3: CANTX -> PWM
- U4 pad 1: Net-(U4-Pad1) -> VIN
- U4 pad 2: GND -> Net-(D1-Pad1)
- U4 pad 3: CLK -> GND
- U4 pad 4: VIO -> Net-(C20-Pad2)
- U5 pad 1: CANRX -> UART_TX
- U5 pad 4: CANTX -> UART_RX
- U6 pad 1: Net-(U6-Pad1) -> +12V
- U6 pad 2: GND -> Net-(C1-Pad1)
- U6 pad 3: GND -> Net-(D3-Pad1)
- U6 pad 4: ENC_A -> U
- U6 pad 5: GND -> UH
- U6 pad 6: ENC_A_A -> UL
- U6 pad 7: ENC_A_B -> GND
- U6 pad 8: +5V -> Net-(D4-Pad1)
- U7 pad 1: Net-(U7-Pad1) -> +12V
- U7 pad 2: GND -> Net-(C11-Pad1)
- U7 pad 3: GND -> Net-(D8-Pad1)
- U7 pad 4: ENC_B -> V
- U7 pad 5: GND -> VH
- U7 pad 6: ENC_B_A -> VL
- U7 pad 7: ENC_B_B -> GND
- U7 pad 8: +5V -> Net-(D9-Pad1)
Routing:
- net +5V: track 162.5 -> 15.4 mm, vias 6 -> 0
- net VIO: track 106.6 -> 0.00 mm, vias 5 -> 0
- net Vin_mon: track 99.7 -> 0.00 mm, vias 2 -> 0
- net VP: track 79.9 -> 0.00 mm, vias 3 -> 0
- net NTC_EXT: track 72.8 -> 0.00 mm, vias 1 -> 0
- net HALL3: track 70.8 -> 0.00 mm, vias 2 -> 0
- net HALL2: track 68.5 -> 0.00 mm, vias 2 -> 0
- net HALL1: track 60.7 -> 0.00 mm, vias 2 -> 0
- net ENC_B: track 54.4 -> 0.00 mm, vias 4 -> 0
- net ENC_A: track 49.3 -> 0.00 mm, vias 4 -> 0
- net VHM: track 46.2 -> 0.00 mm, vias 2 -> 0
- net GND: track 77.8 -> 31.6 mm, vias 103 -> 48
- net CSM: track 44.9 -> 0.00 mm, vias 2 -> 0
- net Net-(C20-Pad1): track 39.6 -> 0.00 mm
- net Net-(D16-Pad2): track 35.1 -> 0.00 mm
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
Commit message: updated files
Parts:
- moved C10 93.6 mm to (13.5, 103.0)
- moved R21 93.0 mm to (25.6, 102.7)
- moved C22 93.0 mm to (54.7, 104.5)
- moved C40 93.0 mm to (25.6, 104.2)
- moved U12 93.0 mm to (47.9, 85.7)
- moved R26 80.6 mm to (45.8, 43.2), turned to 90 degrees
- moved L2 61.3 mm to (39.3, 55.9), turned to 90 degrees
- moved C7 57.2 mm to (31.3, 59.1), turned to 180 degrees
- moved R40 54.4 mm to (56.0, 52.4), turned to 180 degrees
- moved C33 53.8 mm to (39.1, 52.1), turned to 90 degrees
- moved C41 53.8 mm to (41.0, 51.3), turned to 90 degrees
- moved C1 51.4 mm to (50.8, 63.5), turned to 270 degrees
- moved C42 50.1 mm to (61.4, 34.0), turned to 180 degrees
- moved FB1 49.2 mm to (72.9, 39.2)
- moved D1 46.5 mm to (34.8, 54.8)
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Connections:
- Y1 pad 3: GND -> Net-(C4-Pad1)
- Y1 pad 4: Net-(C4-Pad1) -> GND
Routing:
- net GND: track 31.6 -> 25.7 mm, vias 48 -> 41
- net Net-(C3-Pad1): track 5.83 -> 0.00 mm
- net Net-(C13-Pad2): track 5.46 -> 0.00 mm
- net Net-(C14-Pad1): track 4.81 -> 0.00 mm
- net Net-(C2-Pad2): track 3.99 -> 0.00 mm
- net IVH: track 0.00 -> 2.78 mm
- net V: track 2.12 -> 0.00 mm
- net VIN: track 5.87 -> 3.80 mm
- net UU: track 0.91 -> 0.00 mm, vias 1 -> 0
- net U: track 0.81 -> 0.00 mm

Commit message: updated files
Parts:
- moved C43 92.8 mm to (45.0, 79.6), turned to 180 degrees
- moved D2 80.8 mm to (45.9, 49.0), turned to 270 degrees
- moved D5 79.2 mm to (46.1, 61.2), turned to 90 degrees
- moved C20 73.6 mm to (43.6, 59.9)
- moved D7 71.9 mm to (45.5, 36.4), turned to 270 degrees
- moved R7 68.5 mm to (43.6, 58.5), turned to 180 degrees
- moved R1 68.4 mm to (43.6, 61.3), turned to 180 degrees
- moved D13 67.6 mm to (45.5, 31.6), turned to 90 degrees
- moved D10 65.9 mm to (43.2, 31.6), turned to 90 degrees
- moved C38 61.0 mm to (42.4, 51.1)
- moved D6 59.2 mm to (43.2, 36.4), turned to 270 degrees
- moved C22 49.2 mm to (41.6, 57.1)
- moved C25 48.4 mm to (50.6, 46.8), turned to 180 degrees
- moved C33 28.7 mm to (56.9, 74.7), turned to 0 degrees
- moved D1 5.48 mm to (36.5, 60.0), turned to 90 degrees
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
Commit message: updated files
Parts:
- moved R20 97.6 mm to (22.4, 31.1), turned to 270 degrees
- moved Q2 96.2 mm to (27.1, 31.3)
- moved C39 95.0 mm to (22.4, 34.0), turned to 270 degrees
- moved D14 94.5 mm to (-2.67, 39.2), turned to 270 degrees
- moved C10 93.3 mm to (64.2, 24.7), turned to 90 degrees
- moved J10 92.2 mm to (25.9, 26.1)
- moved J9 77.1 mm to (61.8, 63.8)
- moved D15 73.1 mm to (24.2, 31.8), turned to 90 degrees
- moved C40 70.6 mm to (27.1, 33.6), turned to 0 degrees
- moved R21 67.7 mm to (27.1, 35.0), turned to 0 degrees
- moved D17 62.6 mm to (67.1, 26.1), turned to 270 degrees
- moved J11 53.6 mm to (74.5, 25.9)
- moved R39 49.6 mm to (73.5, 34.4), turned to 0 degrees
- moved C28 47.5 mm to (85.6, 9.66)
- moved U12 42.9 mm to (64.9, 46.3)
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Connections:
- U8 pad 6: NTC_EXT -> Net-(U8-Pad6)
- U9 pad 4: Net-(U9-Pad4) -> NTC_EXT
Routing:
- net GND: track 25.7 -> 13.7 mm, vias 41 -> 25
- net Net-(C40-Pad1): track 10.5 -> 0.00 mm, vias 1 -> 0
- net NTC_EXT_GND: track 4.69 -> 0.00 mm
- net SK6812_OUT: track 2.82 -> 0.00 mm

Commit message: updated files
Parts:
- added C50: 10nF, Capacitor_SMD:C_0805_2012Metric, F.Cu at (43.6, 65.6)
- added C51: 10nF, Capacitor_SMD:C_0805_2012Metric, F.Cu at (45.2, 45.0)
- added C52: 10nF, Capacitor_SMD:C_0805_2012Metric, F.Cu at (40.9, 35.4)
- added R18: 1, Resistor_SMD:R_0603_1608Metric, F.Cu at (45.9, 64.6)
- added R22: 1, Resistor_SMD:R_0603_1608Metric, F.Cu at (46.0, 42.7)
- added R43: 1, Resistor_SMD:R_0603_1608Metric, F.Cu at (47.5, 35.5)
- R27, R28, R29: value 100 -> 1.8k
- R33, R34, R35: value 1k -> 10k
- moved C28 44.9 mm to (41.3, 16.7)
- moved C37 35.5 mm to (38.9, 43.7)
- moved C27 35.5 mm to (34.0, 47.7)
- moved C35 35.5 mm to (36.6, 44.3)
- moved C36 35.5 mm to (40.7, 43.7)
- moved D14 35.5 mm to (32.2, 46.1)
- moved L1 35.5 mm to (35.8, 41.2)
- moved R37 35.5 mm to (41.3, 47.6)
- moved R38 35.5 mm to (39.7, 47.6)
- moved U3 35.5 mm to (36.9, 47.0)
- moved R26 3.33 mm to (44.1, 40.3)
- moved C20 2.79 mm to (43.6, 62.7)
- moved C22 2.79 mm to (41.6, 59.9)
- moved C23 2.79 mm to (42.4, 58.2)
- moved C38 2.79 mm to (42.4, 53.9)
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Connections:
- C27 pad 1: VP -> +12V
- J9 pad 1: VIO -> +3V3
- JP2 pad 1: VIO -> +3V3
- P1 pad 1: VIO -> +3V3
- R33 pad 1: VIO -> +3V3
- R34 pad 1: VIO -> +3V3
- R35 pad 1: VIO -> +3V3
- R46 pad 1: VIO -> +3V3
- U3 pad 2: VP -> +12V
Routing:
- net GND: vias 25 -> 24
- removed copper zone on F.Cu, net GND

Commit message: updated files
Parts:
- moved C28 40.6 mm to (75.3, 39.0), turned to 90 degrees
- moved D2 0.52 mm to (45.7, 49.4)
- moved D5 0.34 mm to (43.4, 49.1)
- moved R43 0.28 mm to (47.3, 35.8)
- moved R31 0.16 mm to (45.7, 27.8)
- moved R30 0.16 mm to (45.7, 25.0)
- moved D1 0.11 mm to (36.6, 62.8)
- moved R24 0.11 mm to (45.7, 57.4)
Connections:
- U8 pad 3: SWDCL -> SWCLK
Routing:
- net +12V: track 0.00 -> 133.4 mm, vias 0 -> 23
- net GND: track 13.7 -> 63.3 mm, vias 24 -> 23
- net Vin_mon: track 0.00 -> 44.3 mm
- net +3V3: track 0.00 -> 35.9 mm
- net NTC_EXT: track 0.00 -> 35.6 mm
- net VIN: track 3.80 -> 23.7 mm
- net U: track 0.00 -> 19.9 mm
- net W: track 0.00 -> 19.4 mm
- net V: track 0.00 -> 19.2 mm
- net SWCLK: track 0.00 -> 17.8 mm
- net Net-(D3-Pad1): track 0.00 -> 15.1 mm
- net SWDIO: track 0.00 -> 14.8 mm
- net HALL1: track 0.00 -> 14.6 mm
- net UART_TX: track 0.00 -> 12.4 mm
- net Net-(C20-Pad2): track 0.00 -> 11.3 mm, vias 0 -> 2
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
Commit message: updated files
Parts:
- moved C29 12.3 mm to (73.5, 35.8), turned to 0 degrees
- moved C31 12.3 mm to (61.4, 37.1), turned to 180 degrees
- moved R36 10.7 mm to (59.1, 33.4), turned to 270 degrees
- moved R9 10.6 mm to (66.5, 41.1), turned to 90 degrees
- moved R8 10.0 mm to (67.8, 41.1)
- moved R16 9.98 mm to (59.1, 36.2)
- moved C44 6.67 mm to (67.2, 39.0)
- moved C19 6.62 mm to (61.4, 35.8)
- moved R24 0.12 mm to (45.8, 57.4)
- turned R26 to 270 degrees
Connections:
- C26 pad 1: +3V3 -> +5V
- U1 pad 11: IUL -> IWL
- U1 pad 12: UU -> UW
- U1 pad 17: IWH -> IUH
- U1 pad 19: IWL -> IUL
- U1 pad 2: UL -> WL
- U1 pad 24: UW -> UU
- U1 pad 28: WL -> UL
- U1 pad 30: UH -> WH
- U1 pad 32: WH -> UH
- U1 pad 44: HALL1 -> HALL3
- U1 pad 46: HALL3 -> HALL1
- U1 pad 9: IUH -> IWH
Routing:
- net +5V: track 5.31 -> 117.2 mm, vias 0 -> 8
- net +3V3: track 35.9 -> 145.5 mm, vias 0 -> 8
- net Vin_mon: track 44.3 -> 89.7 mm, vias 0 -> 2
- net HALL3: track 1.70 -> 45.7 mm, vias 0 -> 2
- net HALL2: track 7.48 -> 48.2 mm, vias 0 -> 2
- net HALL1: track 14.6 -> 53.9 mm, vias 0 -> 2
- net UV: track 2.99 -> 30.6 mm, vias 0 -> 2
- net WH: track 0.00 -> 24.9 mm, vias 0 -> 2
- net UW: track 9.23 -> 33.0 mm, vias 0 -> 2
- net IWH: track 5.39 -> 28.1 mm
- net UU: track 2.91 -> 24.3 mm, vias 0 -> 2
- net GPIO_BEMF: track 1.43 -> 22.3 mm, vias 0 -> 1
- net SK6812: track 0.00 -> 12.8 mm, vias 0 -> 2
- net IWL: track 3.72 -> 16.2 mm, vias 0 -> 2
- net WL: track 0.00 -> 11.7 mm, vias 0 -> 2
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- added copper zone on F.Cu, net +3V3
- added copper zone on F.Cu, net GND

Commit message: updated files
Parts:
- removed C34: 100n, Capacitor_SMD:C_0603_1608Metric
- moved R21 3.42 mm to (23.8, 35.6), turned to 270 degrees
- moved C40 2.80 mm to (25.1, 35.6), turned to 270 degrees
Routing:
- net NTC_EXT: track 36.8 -> 89.2 mm, vias 1 -> 2
- net CANTX: track 1.46 -> 48.1 mm, vias 1 -> 4
- net UL: track 1.30 -> 47.9 mm, vias 1 -> 3
- net UH: track 5.33 -> 50.0 mm, vias 1 -> 2
- net PWM: track 3.15 -> 44.6 mm, vias 1 -> 3
- net VH: track 5.22 -> 43.0 mm, vias 1 -> 2
- net UART_RX: track 12.0 -> 49.7 mm, vias 1 -> 2
- net CANRX: track 5.16 -> 40.1 mm, vias 1 -> 2
- net UART_TX: track 15.7 -> 49.3 mm, vias 1 -> 2
- net RS485RXTX: track 4.96 -> 38.1 mm, vias 1 -> 2
- net GPIO_BEMF: track 22.3 -> 52.0 mm, vias 1 -> 2
- net VL: track 1.32 -> 30.2 mm, vias 1 -> 2
- net Ain: track 1.12 -> 28.0 mm, vias 1 -> 2
- net UU: track 24.3 -> 48.4 mm, vias 2 -> 3
- net IUL: track 4.23 -> 25.9 mm
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