File: STM32G431/PAC5523.kicad_pcb (KiCad board)
At the start: 4 copper layers, 60 x 44 mm, 141 parts, among them J1 W, J10 NTC, J11 LED, J2 U, J3 V, J4 GND, J5 VIN, J6 UART, J8 HALL, J9 AIN/PWM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

Commit message: updated files
Routing:
- net GPIO_BEMF: track 52.0 -> 47.1 mm
- net UW: track 33.0 -> 34.9 mm
- net VDDA: track 8.40 -> 6.64 mm
- net IWL: track 16.2 -> 14.6 mm
- net +3V3: track 151.3 -> 149.7 mm
- net IUL: track 25.9 -> 26.7 mm
- net CANTX: track 48.1 -> 48.9 mm
- net HALL1: track 53.6 -> 54.1 mm
Other:
- board text added: "CPU STM32G431"
- board text added: "GND AIN PWM 3.3V"
- board text added: "GND H3 H2 H1 5V"
- board text added: "UART/CAN/RS485 ANALOG/PWM/ENCODER"
- board text removed: "CPU 1"
- board text removed: "GND AIN 3.3V"
- board text removed: "GND B- B+ A- A+ +5V"
- board text removed: "GND H3 H2 H1 VIO"
- board text removed: "OttercontrolNG"
- board text removed: "UART/CAN/RS485 ANALOG/ENCODER"

Commit message: updated files
Parts:
- added C34: 100n, Capacitor_SMD:C_0603_1608Metric, F.Cu at (5.91, 42.0)
- added C53: 10u, Capacitor_SMD:C_1206_3216Metric, F.Cu at (2.66, 35.8)
- added D16: LED, Diode_SMD:D_0603_1608Metric, F.Cu at (1.90, 42.1)
- added D18: LED, Diode_SMD:D_0603_1608Metric, F.Cu at (10.8, 39.8)
- added D19: LED, Diode_SMD:D_0603_1608Metric, F.Cu at (26.3, 33.6)
- added R44: 10, Resistor_SMD:R_1206_3216Metric, F.Cu at (34.0, 62.9)
- added R47: 22k, Resistor_SMD:R_0603_1608Metric, F.Cu at (15.3, 40.8)
- added R48: 22k, Resistor_SMD:R_0603_1608Metric, F.Cu at (6.67, 45.9)
- added R49: 22k, Resistor_SMD:R_0603_1608Metric, F.Cu at (10.7, 45.9)
- added R50: 10, Resistor_SMD:R_1206_3216Metric, F.Cu at (11.6, 36.9)
- L2: footprint Inductor_SMD:L_Taiyo-Yuden_MD-4040 -> Inductor_SMD:L_Taiyo-Yuden_MD-5050
Connections:
- C21 pad 1: VIN -> Net-(C21-Pad1)
- C7 pad 1: VIN -> Net-(C21-Pad1)
- U4 pad 1: VIN -> Net-(C21-Pad1)
Routing:
- net Net-(C21-Pad1): track 0.00 -> 8.25 mm
- net Net-(C20-Pad2): track 11.3 -> 13.4 mm
- net VIN: track 23.7 -> 21.8 mm
- net GND: vias 152 -> 151

Commit message: updated pcb
Parts:
- removed C34: 100n, Capacitor_SMD:C_0603_1608Metric
- C22, C43, C46: value 100n 100V -> 100n
- D1: value SM4007PL -> SS310; footprint Diode_SMD:D_SOD-123F -> Diode_SMD:D_SMA
- R47: value 22k -> 2k
- R48: value 22k -> 1k
- R49: value 22k -> 660
- U1: footprint Package_DFN_QFN:QFN-48-1EP_6x6mm_P0.4mm_EP4.2x4.2mm -> Package_DFN_QFN:QFN-48-1EP_7x7mm_P0.5mm_EP5.3x5.3mm
- moved C53 37.3 mm to (37.8, 48.4), turned to 180 degrees
- moved R50 32.6 mm to (41.2, 50.6), turned to 270 degrees
- moved R48 25.4 mm to (31.3, 39.7)
- moved D16 24.7 mm to (26.4, 39.5)
- moved R49 21.9 mm to (31.3, 38.4)
- moved R47 15.9 mm to (31.3, 41.1)
- moved D18 15.7 mm to (26.4, 38.1)
- moved R44 7.43 mm to (26.9, 65.1), turned to 0 degrees
- moved D1 4.13 mm to (32.8, 64.5), turned to 180 degrees
- moved R21 3.95 mm to (27.5, 34.4)
- moved D19 3.06 mm to (26.4, 36.7)
- moved C21 2.61 mm to (33.6, 61.5), turned to 0 degrees
- moved C7 2.21 mm to (30.9, 59.5)
- moved C37 1.82 mm to (38.9, 41.9)
- moved R37 1.82 mm to (41.3, 45.8)
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Routing:
- net +12V: track 136.3 -> 147.4 mm
- net VIN: track 21.8 -> 13.0 mm
- net Net-(C21-Pad1): track 8.25 -> 16.7 mm
- net Net-(D1-Pad1): track 8.78 -> 13.6 mm
- net Net-(D16-Pad2): track 0.00 -> 3.95 mm
- net Net-(D19-Pad2): track 0.00 -> 3.95 mm
- net Net-(D18-Pad2): track 0.00 -> 3.93 mm
- net +3V3: track 149.7 -> 153.5 mm
- net +5V: track 130.6 -> 134.1 mm
- net Net-(C53-Pad1): track 0.00 -> 2.35 mm
- net UW: track 34.9 -> 32.9 mm
- net UL: track 47.9 -> 46.7 mm
- net NTC_IO: track 3.27 -> 2.29 mm
- net GPIO_BEMF: track 47.1 -> 46.2 mm
- net VDDA: track 6.64 -> 5.73 mm
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Other:
- board text added: "+12V"
- board text added: "+3.3V"
- board text added: "+5.0V"
