File: STM32G431/PAC5523.sch (KiCad schematic (older format))
At the start: 77 parts, among them J1 W, J2 U, J3 V, U1 PAC5523

Commit message: updated files
Parts:
- removed C4, C5: 100n, Capacitor_SMD:C_0603_1608Metric, symbol Device:C_Small
- removed C6, C7: 4u7, Capacitor_SMD:C_0603_1608Metric, symbol Device:C_Small
- removed U1: PAC5523, Package_DFN_QFN:QFN-48-1EP_6x6mm_P0.4mm_EP4.2x4.2mm, symbol otter:PAC5523
- added C? (x3): 4u7, Capacitor_SMD:C_0603_1608Metric, symbol Device:C_Small
- C7: renamed from C?; footprint (none) -> Capacitor_THT:CP_Radial_D8.0mm_P3.80mm
- D1: renamed from D?; value SS310 -> SM4007PL
- D11, D12, D3, D4, D9: value SS310 -> SM4007PL
- D8: value SS310 -> SM4007PL; LCSC (none) -> C64898
- FB1: renamed from FB?; footprint (none) -> Inductor_SMD:L_0805_2012Metric
- L2: renamed from L?; footprint (none) -> Inductor_SMD:L_Taiyo-Yuden_MD-4040
- U1: renamed from U?; footprint (none) -> Package_DFN_QFN:QFN-48-1EP_6x6mm_P0.4mm_EP4.2x4.2mm
- U10, U6, U7: renamed from U?; footprint (none) -> Package_SO:SOIC-8_3.9x4.9mm_P1.27mm
- Y1: renamed from Y?; footprint (none) -> Crystal:Crystal_SMD_3225-4Pin_3.2x2.5mm
- gave numbers to parts that had none: 30
Connections:
- net VIO is gone; now on net +3V3: C8.1
- net +12V: now also U10.1 (VDD), U6.1 (VDD), U7.1 (VDD), C?.1, C?.1, C?.1
- net +3V3: now also C9.1
- net Ain: now also U1.25 (PB12)
- net CANRX: now also U1.33 (PA11)
- net CANTX: now also U1.47 (PB9)
- net GND: now also U10.7 (VSS), U6.7 (VSS), U7.7 (VSS), C?.2, C?.2, C?.2
- net NTC_IO: now also U1.27 (PB14)
- net RS485RXTX: now also U1.40 (PC11)
- net SK6812: now also U1.29 (PC6)
- net UH: now also U6.5 (HI)
- net UL: now also U6.6 (LI)
- net VH: now also U7.5 (HI)
- net VL: now also U7.6 (LI)
- net Vin_mon: now also U1.8 (PA0)
- net WH: now also U10.5 (HI)
- net WL: now also U10.6 (LI)
- net PWM: now reaches U1.38 (PA15)
- net UART_TX: now reaches U1.41 (PB3)
- net UART_RX: now reaches U1.42 (PB4)
- net GPIO_BEMF: now reaches U1.43 (PB5)
Other:
- moved on the sheet: C10, C24, C25, C26, C28, C32, C33, C34, C8, C9

Commit message: updated files
Parts:
- Y1: symbol Device:Crystal_GND23_Small -> Device:Crystal_GND24
- gave numbers to parts that had none: 3
Connections:
- net GND: now also Y1.4; no longer Y1.3
- net at C4.1, U1.5 (PF0-OSC_IN): now also Y1.3; no longer Y1.4
Other:
- moved on the sheet: C4, C5
Changed lines of the file:
@@
 $EndComp
-$Comp
-L Device:Crystal_GND23_Small Y1
-U 1 1 5DD492E5
-P 2050 3100
-F 0 "Y1" H 1850 2800 50  0000 C CNN
-F 1 "8Mhz" H 1850 2900 50  0000 C CNN
-F 2 "Crystal:Crystal_SMD_3225-4Pin_3.2x2.5mm" H 2050 3100 50  0001 C CNN
-F 3 "~" H 2050 3100 50  0001 C CNN
-	1    2050 3100
-	-1   0    0    1
-$EndComp
-Wire Wire Line
-	1950 2950 1950 3100
 $Comp
 L power:GND #PWR0114
 U 1 1 5DDB4600
-P 2200 3300
-F 0 "#PWR0114" H 2200 3050 50  0001 C CNN
-F 1 "GND" H 2205 3127 50  0000 C CNN
-F 2 "" H 2200 3300 50  0001 C CNN
-F 3 "" H 2200 3300 50  0001 C CNN
-	1    2200 3300
-	1    0    0    -1
-$EndComp
-Wire Wire Line
-	1950 2950 2700 2950
+P 1900 3500
+F 0 "#PWR0114" H 1900 3250 50  0001 C CNN
+F 1 "GND" H 1905 3327 50  0000 C CNN
+F 2 "" H 1900 3500 50  0001 C CNN
+F 3 "" H 1900 3500 50  0001 C CNN
+	1    1900 3500
+	1    0    0    -1
+$EndComp
 $Comp
 L power:GND #PWR0116
 U 1 1 5DDE1D7B
-P 1900 3300
-F 0 "#PWR0116" H 1900 3050 50  0001 C CNN
-F 1 "GND" H 1905 3127 50  0000 C CNN
-F 2 "" H 1900 3300 50  0001 C CNN
-F 3 "" H 1900 3300 50  0001 C CNN
-	1    1900 3300
-	1    0    0    -1
+P 1900 2600
+F 0 "#PWR0116" H 1900 2350 50  0001 C CNN
+F 1 "GND" H 1905 2427 50  0000 C CNN
+F 2 "" H 1900 2600 50  0001 C CNN
+F 3 "" H 1900 2600 50  0001 C CNN
+	1    1900 2600
+	-1   0    0    1
 $EndComp
 $Comp
 L Device:C_Small C5
 U 1 1 5DDF34E1
-P 2200 3200
-F 0 "C5" H 2292 3246 50  0000 L CNN
-F 1 "18p" H 2292 3155 50  0000 L CNN
-F 2 "Capacitor_SMD:C_0603_1608Metric" H 2200 3200 50  0001 C CNN
-F 3 "~" H 2200 3200 50  0001 C CNN
-	1    2200 3200
+P 1900 3400
+F 0 "C5" H 1992 3446 50  0000 L CNN
+F 1 "18p" H 1992 3355 50  0000 L CNN
+F 2 "Capacitor_SMD:C_0603_1608Metric" H 1900 3400 50  0001 C CNN
+F 3 "~" H 1900 3400 50  0001 C CNN
+	1    1900 3400
 	1    0    0    -1
 $EndComp
@@
 L Device:C_Small C4
 U 1 1 5DDFCA58
-P 1900 3200
-F 0 "C4" H 1808 3246 50  0000 R CNN
-F 1 "18p" H 1808 3155 50  0000 R CNN
-F 2 "Capacitor_SMD:C_0603_1608Metric" H 1900 3200 50  0001 C CNN
-F 3 "~" H 1900 3200 50  0001 C CNN
-	1    1900 3200
-	1    0    0    -1
-$EndComp
-Wire Wire Line
-	1950 3100 1900 3100
-Connection ~ 1950 3100
-Wire Wire Line
-	2150 3100 2200 3100
-Wire Wire Line
-	2200 3100 2700 3100
-Connection ~ 2200 3100
+P 1900 2700
+F 0 "C4" H 1808 2746 50  0000 R CNN
+F 1 "18p" H 1808 2655 50  0000 R CNN
+F 2 "Capacitor_SMD:C_0603_1608Metric" H 1900 2700 50  0001 C CNN
+F 3 "~" H 1900 2700 50  0001 C CNN
+	1    1900 2700
+	-1   0    0    1
+$EndComp
 $Comp
 L power:GND #PWR0117
 U 1 1 5DE39958
-P 2050 3200
-F 0 "#PWR0117" H 2050 2950 50  0001 C CNN
-F 1 "GND" H 2055 3027 50  0000 C CNN
-F 2 "" H 2050 3200 50  0001 C CNN
-F 3 "" H 2050 3200 50  0001 C CNN
-	1    2050 3200
-	1    0    0    -1
+P 1700 3050
+F 0 "#PWR0117" H 1700 2800 50  0001 C CNN
+F 1 "GND" V 1705 2922 50  0000 R CNN
+F 2 "" H 1700 3050 50  0001 C CNN
+F 3 "" H 1700 3050 50  0001 C CNN
+	1    1700 3050
+	0    1    1    0
 $EndComp
 $Comp
 L power:GND #PWR0118
 U 1 1 5DE44094
-P 2050 2900
-F 0 "#PWR0118" H 2050 2650 50  0001 C CNN
-F 1 "GND" H 2055 2727 50  0000 C CNN
-F 2 "" H 2050 2900 50  0001 C CNN
-F 3 "" H 2050 2900 50  0001 C CNN
-	1    2050 2900
-	-1   0    0    1
-$EndComp
-Wire Wire Line
-	2050 3000 2050 2900
+P 2100 3050
+F 0 "#PWR0118" H 2100 2800 50  0001 C CNN
+F 1 "GND" V 2105 2922 50  0000 R CNN
+F 2 "" H 2100 3050 50  0001 C CNN
+F 3 "" H 2100 3050 50  0001 C CNN
+	1    2100 3050
+	0    -1   -1   0
+$EndComp
 $Comp
 L Device:C_Small C18
@@
 $EndComp
 $Comp
-L power:GND #PWR?
+L power:GND #PWR0180
 U 1 1 5DD27A36
 P 7650 5050
-F 0 "#PWR?" H 7650 4800 50  0001 C CNN
+F 0 "#PWR0180" H 7650 4800 50  0001 C CNN
 F 1 "GND" H 7655 4877 50  0000 C CNN
 F 2 "" H 7650 5050 50  0001 C CNN
@@
 $EndComp
 $Comp
-L Device:C_Small C?
+L Device:C_Small C49
 U 1 1 5DD27A3C
 P 7650 4950
-F 0 "C?" H 7742 4996 50  0000 L CNN
+F 0 "C49" H 7742 4996 50  0000 L CNN
 F 1 "4u7" H 7742 4905 50  0000 L CNN
 F 2 "Capacitor_SMD:C_0603_1608Metric" H 7650 4950 50  0001 C CNN
@@
 	7650 4800 7650 4850
 $Comp
-L power:GND #PWR?
+L power:GND #PWR0187
 U 1 1 5DD3E501
 P 7650 3200
-F 0 "#PWR?" H 7650 2950 50  0001 C CNN
+F 0 "#PWR0187" H 7650 2950 50  0001 C CNN
 F 1 "GND" H 7655 3027 50  0000 C CNN
 F 2 "" H 7650 3200 50  0001 C CNN
@@
 $EndComp
 $Comp
-L Device:C_Small C?
+L Device:C_Small C48
 U 1 1 5DD3E507
 P 7650 3100
-F 0 "C?" H 7742 3146 50  0000 L CNN
+F 0 "C48" H 7742 3146 50  0000 L CNN
 F 1 "4u7" H 7742 3055 50  0000 L CNN
 F 2 "Capacitor_SMD:C_0603_1608Metric" H 7650 3100 50  0001 C CNN
@@
 	7650 2950 7650 3000
 $Comp
-L power:GND #PWR?
+L power:GND #PWR0189
 U 1 1 5DD499E9
 P 7650 1350
-F 0 "#PWR?" H 7650 1100 50  0001 C CNN
+F 0 "#PWR0189" H 7650 1100 50  0001 C CNN
 F 1 "GND" H 7655 1177 50  0000 C CNN
 F 2 "" H 7650 1350 50  0001 C CNN
@@
 $EndComp
 $Comp
-L Device:C_Small C?
+L Device:C_Small C47
 U 1 1 5DD499EF
 P 7650 1250
-F 0 "C?" H 7742 1296 50  0000 L CNN
+F 0 "C47" H 7742 1296 50  0000 L CNN
 F 1 "4u7" H 7742 1205 50  0000 L CNN
 F 2 "Capacitor_SMD:C_0603_1608Metric" H 7650 1250 50  0001 C CNN
@@
 Wire Wire Line
 	7650 1100 7650 1150
+$Comp
+L Device:Crystal_GND24 Y1
+U 1 1 5DD492E5
+P 1900 3050
+F 0 "Y1" V 1946 2806 50  0000 R CNN
+F 1 "8Mhz" V 1855 2806 50  0000 R CNN
+F 2 "Crystal:Crystal_SMD_3225-4Pin_3.2x2.5mm" H 1900 3050 50  0001 C CNN
+F 3 "~" H 1900 3050 50  0001 C CNN
+	1    1900 3050
+	0    -1   -1   0
+$EndComp
+Wire Wire Line
+	2700 2950 2650 2950
+Wire Wire Line
+	1900 2850 1900 2900
+Wire Wire Line
+	1900 2850 1900 2800
+Connection ~ 1900 2850
+Wire Wire Line
+	1900 3300 1900 3250
+Connection ~ 1900 3250
+Wire Wire Line
+	1900 3250 1900 3200
+Wire Wire Line
+	2650 3250 2650 3100
+Wire Wire Line
+	2650 3100 2700 3100
+Wire Wire Line
+	2650 2950 2650 2850
+Wire Wire Line
+	1900 2850 2650 2850
+Wire Wire Line
+	1900 3250 2650 3250
 $EndSCHEMATC

Commit message: updated files
Parts:
- C7: LCSC (none) -> C106678
Changed lines of the file:
@@
 F 2 "Capacitor_THT:CP_Radial_D8.0mm_P3.80mm" H 4300 -1350 50  0001 C CNN
 F 3 "~" H 4300 -1350 50  0001 C CNN
+F 4 "C106678" H 4300 -1350 50  0001 C CNN "LCSC"
 	1    4300 -1350
 	1    0    0    -1

Commit message: updated files
Parts:
- added C? (x3): 10nF, Capacitor_SMD:C_0805_2012Metric, symbol Device:C_Small
- added R? (x3): 1, Resistor_SMD:R_0603_1608Metric, symbol Device:R_Small
Connections:
- net GND: now also C?.1, C?.1, C?.1
- net U: now also R?.2
- net V: now also R?.2
- net W: now also R?.2
- new net: C?.2, R?.1 (x3)
Changed lines of the file:
@@
 Text GLabel 4600 4450 2    50   Input ~ 0
 UW
-Text GLabel -100 3600 2    50   Input ~ 0
-Ain
 $Comp
 L Device:C_Small C34
@@
 Wire Wire Line
 	1900 3250 2650 3250
+$Comp
+L Device:R_Small R?
+U 1 1 5DF08F24
+P 10450 1100
+F 0 "R?" V 10346 1100 50  0000 C CNN
+F 1 "1" V 10255 1100 50  0000 C CNN
+F 2 "Resistor_SMD:R_0603_1608Metric" H 10450 1100 50  0001 C CNN
+F 3 "~" H 10450 1100 50  0001 C CNN
+	1    10450 1100
+	1    0    0    -1
+$EndComp
+$Comp
+L Device:C_Small C?
+U 1 1 5DF3323C
+P 10450 900
+F 0 "C?" H 10542 946 50  0000 L CNN
+F 1 "10nF" H 10542 855 50  0000 L CNN
+F 2 "Capacitor_SMD:C_0805_2012Metric" H 10450 900 50  0001 C CNN
+F 3 "~" H 10450 900 50  0001 C CNN
+	1    10450 900
+	1    0    0    -1
+$EndComp
+Wire Wire Line
+	10450 1250 10450 1200
+Connection ~ 10450 1250
+$Comp
+L power:GND #PWR?
+U 1 1 5DF4CD1E
+P 10450 800
+F 0 "#PWR?" H 10450 550 50  0001 C CNN
+F 1 "GND" H 10455 627 50  0000 C CNN
+F 2 "" H 10450 800 50  0001 C CNN
+F 3 "" H 10450 800 50  0001 C CNN
+	1    10450 800
+	-1   0    0    1
+$EndComp
+$Comp
+L Device:R_Small R?
+U 1 1 5DF50507
+P 10450 2950
+F 0 "R?" V 10346 2950 50  0000 C CNN
+F 1 "1" V 10255 2950 50  0000 C CNN
+F 2 "Resistor_SMD:R_0603_1608Metric" H 10450 2950 50  0001 C CNN
+F 3 "~" H 10450 2950 50  0001 C CNN
+	1    10450 2950
+	1    0    0    -1
+$EndComp
+$Comp
+L Device:C_Small C?
+U 1 1 5DF5050D
+P 10450 2750
+F 0 "C?" H 10542 2796 50  0000 L CNN
+F 1 "10nF" H 10542 2705 50  0000 L CNN
+F 2 "Capacitor_SMD:C_0805_2012Metric" H 10450 2750 50  0001 C CNN
+F 3 "~" H 10450 2750 50  0001 C CNN
+	1    10450 2750
+	1    0    0    -1
+$EndComp
+$Comp
+L power:GND #PWR?
+U 1 1 5DF50513
+P 10450 2650
+F 0 "#PWR?" H 10450 2400 50  0001 C CNN
+F 1 "GND" H 10455 2477 50  0000 C CNN
+F 2 "" H 10450 2650 50  0001 C CNN
+F 3 "" H 10450 2650 50  0001 C CNN
+	1    10450 2650
+	-1   0    0    1
+$EndComp
+Wire Wire Line
+	10450 3050 10450 3100
+Connection ~ 10450 3100
+$Comp
+L Device:R_Small R?
+U 1 1 5DF690C9
+P 10450 4800
+F 0 "R?" V 10346 4800 50  0000 C CNN
+F 1 "1" V 10255 4800 50  0000 C CNN
+F 2 "Resistor_SMD:R_0603_1608Metric" H 10450 4800 50  0001 C CNN
+F 3 "~" H 10450 4800 50  0001 C CNN
+	1    10450 4800
+	1    0    0    -1
+$EndComp
+$Comp
+L Device:C_Small C?
+U 1 1 5DF690CF
+P 10450 4600
+F 0 "C?" H 10542 4646 50  0000 L CNN
+F 1 "10nF" H 10542 4555 50  0000 L CNN
+F 2 "Capacitor_SMD:C_0805_2012Metric" H 10450 4600 50  0001 C CNN
+F 3 "~" H 10450 4600 50  0001 C CNN
+	1    10450 4600
+	1    0    0    -1
+$EndComp
+$Comp
+L power:GND #PWR?
+U 1 1 5DF690D5
+P 10450 4500
+F 0 "#PWR?" H 10450 4250 50  0001 C CNN
+F 1 "GND" H 10455 4327 50  0000 C CNN
+F 2 "" H 10450 4500 50  0001 C CNN
+F 3 "" H 10450 4500 50  0001 C CNN
+	1    10450 4500
+	-1   0    0    1
+$EndComp
+Wire Wire Line
+	10450 4900 10450 4950
+Connection ~ 10450 4950
 $EndSCHEMATC

Commit message: updated files
Parts:
- gave numbers to parts that had none: 6
Changed lines of the file:
@@
 	1900 3250 2650 3250
 $Comp
-L Device:R_Small R?
+L Device:R_Small R18
 U 1 1 5DF08F24
 P 10450 1100
-F 0 "R?" V 10346 1100 50  0000 C CNN
+F 0 "R18" V 10346 1100 50  0000 C CNN
 F 1 "1" V 10255 1100 50  0000 C CNN
 F 2 "Resistor_SMD:R_0603_1608Metric" H 10450 1100 50  0001 C CNN
@@
 $EndComp
 $Comp
-L Device:C_Small C?
+L Device:C_Small C50
 U 1 1 5DF3323C
 P 10450 900
-F 0 "C?" H 10542 946 50  0000 L CNN
+F 0 "C50" H 10542 946 50  0000 L CNN
 F 1 "10nF" H 10542 855 50  0000 L CNN
 F 2 "Capacitor_SMD:C_0805_2012Metric" H 10450 900 50  0001 C CNN
@@
 Connection ~ 10450 1250
 $Comp
-L power:GND #PWR?
+L power:GND #PWR0218
 U 1 1 5DF4CD1E
 P 10450 800
-F 0 "#PWR?" H 10450 550 50  0001 C CNN
+F 0 "#PWR0218" H 10450 550 50  0001 C CNN
 F 1 "GND" H 10455 627 50  0000 C CNN
 F 2 "" H 10450 800 50  0001 C CNN
@@
 $EndComp
 $Comp
-L Device:R_Small R?
+L Device:R_Small R22
 U 1 1 5DF50507
 P 10450 2950
-F 0 "R?" V 10346 2950 50  0000 C CNN
+F 0 "R22" V 10346 2950 50  0000 C CNN
 F 1 "1" V 10255 2950 50  0000 C CNN
 F 2 "Resistor_SMD:R_0603_1608Metric" H 10450 2950 50  0001 C CNN
@@
 $EndComp
 $Comp
-L Device:C_Small C?
+L Device:C_Small C51
 U 1 1 5DF5050D
 P 10450 2750
-F 0 "C?" H 10542 2796 50  0000 L CNN
+F 0 "C51" H 10542 2796 50  0000 L CNN
 F 1 "10nF" H 10542 2705 50  0000 L CNN
 F 2 "Capacitor_SMD:C_0805_2012Metric" H 10450 2750 50  0001 C CNN
@@
 $EndComp
 $Comp
-L power:GND #PWR?
+L power:GND #PWR0219
 U 1 1 5DF50513
 P 10450 2650
-F 0 "#PWR?" H 10450 2400 50  0001 C CNN
+F 0 "#PWR0219" H 10450 2400 50  0001 C CNN
 F 1 "GND" H 10455 2477 50  0000 C CNN
 F 2 "" H 10450 2650 50  0001 C CNN
@@
 Connection ~ 10450 3100
 $Comp
-L Device:R_Small R?
+L Device:R_Small R43
 U 1 1 5DF690C9
 P 10450 4800
-F 0 "R?" V 10346 4800 50  0000 C CNN
+F 0 "R43" V 10346 4800 50  0000 C CNN
 F 1 "1" V 10255 4800 50  0000 C CNN
 F 2 "Resistor_SMD:R_0603_1608Metric" H 10450 4800 50  0001 C CNN
@@
 $EndComp
 $Comp
-L Device:C_Small C?
+L Device:C_Small C52
 U 1 1 5DF690CF
 P 10450 4600
-F 0 "C?" H 10542 4646 50  0000 L CNN
+F 0 "C52" H 10542 4646 50  0000 L CNN
 F 1 "10nF" H 10542 4555 50  0000 L CNN
 F 2 "Capacitor_SMD:C_0805_2012Metric" H 10450 4600 50  0001 C CNN
@@
 $EndComp
 $Comp
-L power:GND #PWR?
+L power:GND #PWR0220
 U 1 1 5DF690D5
 P 10450 4500
-F 0 "#PWR?" H 10450 4250 50  0001 C CNN
+F 0 "#PWR0220" H 10450 4250 50  0001 C CNN
 F 1 "GND" H 10455 4327 50  0000 C CNN
 F 2 "" H 10450 4500 50  0001 C CNN

Commit message: updated files
Connections:
- net +3V3: no longer C26.1
- net +5V: now also C26.1
- net HALL1: now also U1.46 (PB8-BOOT0); no longer U1.44 (PB6)
- net HALL3: now also U1.44 (PB6); no longer U1.46 (PB8-BOOT0)
- net IUH: now also U1.17 (PB0); no longer U1.9 (PA1)
- net IUL: now also U1.19 (PB2); no longer U1.11 (PA3)
- net IWH: now also U1.9 (PA1); no longer U1.17 (PB0)
- net IWL: now also U1.11 (PA3); no longer U1.19 (PB2)
- net UH: now also U1.32 (PA10); no longer U1.30 (PA8)
- net UL: now also U1.28 (PB15); no longer U1.2 (PC13)
- net UU: now also U1.24 (PB11); no longer U1.12 (PA4)
- net UW: now also U1.12 (PA4); no longer U1.24 (PB11)
- net WH: now also U1.30 (PA8); no longer U1.32 (PA10)
- net WL: now also U1.2 (PC13); no longer U1.28 (PB15)
Changed lines of the file:
@@
 Wire Wire Line
 	9200 6100 9200 6050
-Text GLabel 4600 4050 2    50   Input ~ 0
+Text GLabel 2700 2200 0    50   Input ~ 0
 HALL1
 Text GLabel 4600 4150 2    50   Input ~ 0
 HALL2
-Text GLabel 4600 3650 2    50   Input ~ 0
-IWL
-Text GLabel 4600 3450 2    50   Input ~ 0
-IWH
 Text GLabel 4600 2250 2    50   Input ~ 0
 IVL
 Text GLabel 4600 2450 2    50   Input ~ 0
 IVH
-Text GLabel 4600 2050 2    50   Input ~ 0
-IUL
-Text GLabel 4600 1850 2    50   Input ~ 0
-IUH
 $Comp
 L Connector:Conn_01x06_Male J2
@@
 Text GLabel 9650 1400 1    50   Input ~ 0
 U
-Text GLabel 4600 2150 2    50   Input ~ 0
-UU
 Text GLabel 2700 4350 0    50   Input ~ 0
 UV
-Text GLabel 4600 4450 2    50   Input ~ 0
-UW
 $Comp
 L Device:C_Small C34
@@
 Text GLabel 2200 1850 0    50   Input ~ 0
 NRST
-Text GLabel 2700 2200 0    50   Input ~ 0
+Text GLabel 4600 4050 2    50   Input ~ 0
 HALL3
 NoConn ~ 2700 2500
@@
 Text GLabel 8500 5100 0    50   Input ~ 0
 WL
-Text GLabel 4600 2550 2    50   Input ~ 0
-UH
-Text GLabel 2700 4750 0    50   Input ~ 0
-UL
 Text GLabel 4600 2650 2    50   Input ~ 0
 VH
 Text GLabel 4600 2950 2    50   Input ~ 0
 VL
-Text GLabel 4600 2750 2    50   Input ~ 0
-WH
-Text GLabel 4600 4850 2    50   Input ~ 0
-WL
 Wire Wire Line
 	10300 5150 10300 5250
@@
 F 3 "" H 5300 7050 50  0001 C CNN
 	1    5300 7050
-	1    0    0    -1
-$EndComp
-$Comp
-L power:+3.3V #PWR0184
-U 1 1 5E77D38A
-P 5650 7050
-F 0 "#PWR0184" H 5650 6900 50  0001 C CNN
-F 1 "+3.3V" H 5665 7223 50  0000 C CNN
-F 2 "" H 5650 7050 50  0001 C CNN
-F 3 "" H 5650 7050 50  0001 C CNN
-	1    5650 7050
 	1    0    0    -1
 $EndComp
@@
 	10450 4900 10450 4950
 Connection ~ 10450 4950
+$Comp
+L power:+5V #PWR?
+U 1 1 5DFF82C4
+P 5650 7050
+AR Path="/5D5C3A79/5DFF82C4" Ref="#PWR?"  Part="1"
+AR Path="/5DFF82C4" Ref="#PWR0184"  Part="1"
+F 0 "#PWR0184" H 5650 6900 50  0001 C CNN
+F 1 "+5V" V 5665 7178 50  0000 L CNN
+F 2 "" H 5650 7050 50  0001 C CNN
+F 3 "" H 5650 7050 50  0001 C CNN
+	1    5650 7050
+	1    0    0    -1
+$EndComp
+Text GLabel 4600 2050 2    50   Input ~ 0
+IWL
+Text GLabel 4600 1850 2    50   Input ~ 0
+IWH
+Text GLabel 4600 2150 2    50   Input ~ 0
+UW
+Text GLabel 4600 2550 2    50   Input ~ 0
+WH
+Text GLabel 4600 2750 2    50   Input ~ 0
+UH
+Text GLabel 4600 3450 2    50   Input ~ 0
+IUH
+Text GLabel 4600 3650 2    50   Input ~ 0
+IUL
+Text GLabel 4600 4450 2    50   Input ~ 0
+UU
+Text GLabel 4600 4850 2    50   Input ~ 0
+UL
+Text GLabel 2700 4750 0    50   Input ~ 0
+WL
 $EndSCHEMATC

Commit message: updated files
Parts:
- added C53: 10u, Capacitor_SMD:C_1206_3216Metric, symbol Device:C_Small
- added D16, D18, D19: LED, Diode_SMD:D_0603_1608Metric, symbol Device:LED
- added R44, R50: 10, Resistor_SMD:R_1206_3216Metric, symbol Device:R
- added R47, R48, R49: 22k, Resistor_SMD:R_0603_1608Metric, symbol Device:R_Small
- L2: footprint Inductor_SMD:L_Taiyo-Yuden_MD-4040 -> Inductor_SMD:L_Taiyo-Yuden_MD-5050
Connections:
- net +12V: now also R47.2, R50.2
- net +3V3: now also R49.2
- net +5V: now also R48.2
- net GND: now also C53.2, D16.1 (K), D18.1 (K), D19.1 (K)
- net VIN: now also R44.1; no longer C21.1, C7.1, U4.1 (VIN)
- new net: C21.1, C7.1, R44.2, U4.1 (VIN)
- new net: D16.2 (A), R47.1
- new net: D18.2 (A), R48.1
- new net: D19.2 (A), R49.1
- new net: C53.1, R50.1
Changed lines of the file:
@@
 	4850 -1450 4300 -1450
 Connection ~ 4850 -1450
-Text GLabel 4300 -1500 1    50   Input ~ 0
+Text GLabel 4300 -1800 1    50   Input ~ 0
 VIN
 Wire Wire Line
@@
 F 0 "L2" V 6940 -1450 50  0000 C CNN
 F 1 "100u 1A" V 6849 -1450 50  0000 C CNN
-F 2 "Inductor_SMD:L_Taiyo-Yuden_MD-4040" H 6750 -1450 50  0001 C CNN
+F 2 "Inductor_SMD:L_Taiyo-Yuden_MD-5050" H 6750 -1450 50  0001 C CNN
 F 3 "~" H 6750 -1450 50  0001 C CNN
 	1    6750 -1450
@@
 Text GLabel 2700 4750 0    50   Input ~ 0
 WL
+$Comp
+L Device:R R44
+U 1 1 5E1B8A15
+P 4300 -1650
+F 0 "R44" H 4370 -1604 50  0000 L CNN
+F 1 "10" H 4370 -1695 50  0000 L CNN
+F 2 "Resistor_SMD:R_1206_3216Metric" V 4230 -1650 50  0001 C CNN
+F 3 "~" H 4300 -1650 50  0001 C CNN
+	1    4300 -1650
+	1    0    0    -1
+$EndComp
+$Comp
+L Device:LED D16
+U 1 1 5E1DA242
+P 3100 7050
+F 0 "D16" V 3139 6933 50  0000 R CNN
+F 1 "LED" V 3048 6933 50  0000 R CNN
+F 2 "Diode_SMD:D_0603_1608Metric" H 3100 7050 50  0001 C CNN
+F 3 "~" H 3100 7050 50  0001 C CNN
+	1    3100 7050
+	0    -1   -1   0
+$EndComp
+$Comp
+L power:GND #PWR0221
+U 1 1 5E1DADD3
+P 3100 7200
+F 0 "#PWR0221" H 3100 6950 50  0001 C CNN
+F 1 "GND" H 3105 7027 50  0000 C CNN
+F 2 "" H 3100 7200 50  0001 C CNN
+F 3 "" H 3100 7200 50  0001 C CNN
+	1    3100 7200
+	1    0    0    -1
+$EndComp
+$Comp
+L Device:R_Small R47
+U 1 1 5E1E1C6C
+P 3100 6800
+F 0 "R47" H 3041 6754 50  0000 R CNN
+F 1 "22k" H 3041 6845 50  0000 R CNN
+F 2 "Resistor_SMD:R_0603_1608Metric" H 3100 6800 50  0001 C CNN
+F 3 "~" H 3100 6800 50  0001 C CNN
+	1    3100 6800
+	-1   0    0    1
+$EndComp
+$Comp
+L Device:LED D18
+U 1 1 5E1EE2BF
+P 3450 7050
+F 0 "D18" V 3489 6933 50  0000 R CNN
+F 1 "LED" V 3398 6933 50  0000 R CNN
+F 2 "Diode_SMD:D_0603_1608Metric" H 3450 7050 50  0001 C CNN
+F 3 "~" H 3450 7050 50  0001 C CNN
+	1    3450 7050
+	0    -1   -1   0
+$EndComp
+$Comp
+L power:GND #PWR0222
+U 1 1 5E1EE2C5
+P 3450 7200
+F 0 "#PWR0222" H 3450 6950 50  0001 C CNN
+F 1 "GND" H 3455 7027 50  0000 C CNN
+F 2 "" H 3450 7200 50  0001 C CNN
+F 3 "" H 3450 7200 50  0001 C CNN
+	1    3450 7200
+	1    0    0    -1
+$EndComp
+$Comp
+L Device:R_Small R48
+U 1 1 5E1EE2CB
+P 3450 6800
+F 0 "R48" H 3391 6754 50  0000 R CNN
+F 1 "22k" H 3391 6845 50  0000 R CNN
+F 2 "Resistor_SMD:R_0603_1608Metric" H 3450 6800 50  0001 C CNN
+F 3 "~" H 3450 6800 50  0001 C CNN
+	1    3450 6800
+	-1   0    0    1
+$EndComp
+$Comp
+L Device:LED D19
+U 1 1 5E1F9EDC
+P 3800 7050
+F 0 "D19" V 3839 6933 50  0000 R CNN
+F 1 "LED" V 3748 6933 50  0000 R CNN
+F 2 "Diode_SMD:D_0603_1608Metric" H 3800 7050 50  0001 C CNN
+F 3 "~" H 3800 7050 50  0001 C CNN
+	1    3800 7050
+	0    -1   -1   0
+$EndComp
+$Comp
+L power:GND #PWR0223
+U 1 1 5E1F9EE2
+P 3800 7200
+F 0 "#PWR0223" H 3800 6950 50  0001 C CNN
+F 1 "GND" H 3805 7027 50  0000 C CNN
+F 2 "" H 3800 7200 50  0001 C CNN
+F 3 "" H 3800 7200 50  0001 C CNN
+	1    3800 7200
+	1    0    0    -1
+$EndComp
+$Comp
+L Device:R_Small R49
+U 1 1 5E1F9EE8
+P 3800 6800
+F 0 "R49" H 3741 6754 50  0000 R CNN
+F 1 "22k" H 3741 6845 50  0000 R CNN
+F 2 "Resistor_SMD:R_0603_1608Metric" H 3800 6800 50  0001 C CNN
+F 3 "~" H 3800 6800 50  0001 C CNN
+	1    3800 6800
+	-1   0    0    1
+$EndComp
+$Comp
+L power:+12V #PWR0224
+U 1 1 5E224619
+P 3100 6700
+F 0 "#PWR0224" H 3100 6550 50  0001 C CNN
+F 1 "+12V" H 3115 6873 50  0000 C CNN
+F 2 "" H 3100 6700 50  0001 C CNN
+F 3 "" H 3100 6700 50  0001 C CNN
+	1    3100 6700
+	1    0    0    -1
+$EndComp
+$Comp
+L power:+3.3V #PWR0225
+U 1 1 5E237284
+P 3800 6700
+F 0 "#PWR0225" H 3800 6550 50  0001 C CNN
+F 1 "+3.3V" H 3815 6873 50  0000 C CNN
+F 2 "" H 3800 6700 50  0001 C CNN
+F 3 "" H 3800 6700 50  0001 C CNN
+	1    3800 6700
+	1    0    0    -1
+$EndComp
+$Comp
+L power:+5V #PWR?
+U 1 1 5E247F17
+P 3450 6700
+AR Path="/5D59ABFE/5E247F17" Ref="#PWR?"  Part="1"
+AR Path="/5E247F17" Ref="#PWR0226"  Part="1"
+F 0 "#PWR0226" H 3450 6550 50  0001 C CNN
+F 1 "+5V" H 3465 6873 50  0000 C CNN
+F 2 "" H 3450 6700 50  0001 C CNN
+F 3 "" H 3450 6700 50  0001 C CNN
+	1    3450 6700
+	1    0    0    -1
+$EndComp
+$Comp
+L Device:R R50
+U 1 1 5E25917B
+P 7950 -1600
+F 0 "R50" H 8020 -1554 50  0000 L CNN
+F 1 "10" H 8020 -1645 50  0000 L CNN
+F 2 "Resistor_SMD:R_1206_3216Metric" V 7880 -1600 50  0001 C CNN
+F 3 "~" H 7950 -1600 50  0001 C CNN
+	1    7950 -1600
+	1    0    0    -1
+$EndComp
+$Comp
+L Device:C_Small C53
+U 1 1 5E26584B
+P 7950 -1850
+F 0 "C53" H 8042 -1804 50  0000 L CNN
+F 1 "10u" H 8042 -1895 50  0000 L CNN
+F 2 "Capacitor_SMD:C_1206_3216Metric" H 7950 -1850 50  0001 C CNN
+F 3 "~" H 7950 -1850 50  0001 C CNN
+	1    7950 -1850
+	-1   0    0    1
+$EndComp
+$Comp
+L power:GND #PWR0227
+U 1 1 5E265851
+P 7950 -1950
+F 0 "#PWR0227" H 7950 -2200 50  0001 C CNN
+F 1 "GND" H 7955 -2123 50  0000 C CNN
+F 2 "" H 7950 -1950 50  0001 C CNN
+F 3 "" H 7950 -1950 50  0001 C CNN
+	1    7950 -1950
+	-1   0    0    1
+$EndComp
 $EndSCHEMATC
