File: STM32G431/STM32G431.sch (KiCad schematic (older format))
At the start: 93 parts, among them J1 W, J2 U, J3 V, U1 STM32G431CBUx, U10 MIC4605, U12 AP2204R-3.3, U4 XL7015, U6 MIC4605, U7 MIC4605, Y1 8Mhz

Commit message: updated files
Parts:
- C44, C45: value 100p -> DNP
- R10, R11, R12, R13, R2, R3: value 2 -> 33
Other:
- moved on the sheet: C43, C46, U12
Changed lines of the file:
@@
 EESchema Schematic File Version 4
-LIBS:STM32G431-cache
 EELAYER 30 0
 EELAYER END
@@
 P 9900 1300
 F 0 "R2" V 9950 1450 50  0000 C CNN
-F 1 "2" V 9900 1300 50  0000 C CNN
+F 1 "33" V 9900 1300 50  0000 C CNN
 F 2 "Resistor_SMD:R_0805_2012Metric" H 9900 1300 50  0001 C CNN
 F 3 "~" H 9900 1300 50  0001 C CNN
@@
 P 9900 1600
 F 0 "R3" V 10004 1600 50  0000 C CNN
-F 1 "2" V 10095 1600 50  0000 C CNN
+F 1 "33" V 10095 1600 50  0000 C CNN
 F 2 "Resistor_SMD:R_0805_2012Metric" H 9900 1600 50  0001 C CNN
 F 3 "~" H 9900 1600 50  0001 C CNN
@@
 P 9900 3150
 F 0 "R10" V 9950 3300 50  0000 C CNN
-F 1 "2" V 9900 3150 50  0000 C CNN
+F 1 "33" V 9900 3150 50  0000 C CNN
 F 2 "Resistor_SMD:R_0805_2012Metric" H 9900 3150 50  0001 C CNN
 F 3 "~" H 9900 3150 50  0001 C CNN
@@
 P 9900 3450
 F 0 "R11" V 10004 3450 50  0000 C CNN
-F 1 "2" V 10095 3450 50  0000 C CNN
+F 1 "33" V 10095 3450 50  0000 C CNN
 F 2 "Resistor_SMD:R_0805_2012Metric" H 9900 3450 50  0001 C CNN
 F 3 "~" H 9900 3450 50  0001 C CNN
@@
 P 9900 5000
 F 0 "R12" V 9950 5150 50  0000 C CNN
-F 1 "2" V 9900 5000 50  0000 C CNN
+F 1 "33" V 9900 5000 50  0000 C CNN
 F 2 "Resistor_SMD:R_0805_2012Metric" H 9900 5000 50  0001 C CNN
 F 3 "~" H 9900 5000 50  0001 C CNN
@@
 P 9900 5300
 F 0 "R13" V 10004 5300 50  0000 C CNN
-F 1 "2" V 10095 5300 50  0000 C CNN
+F 1 "33" V 10095 5300 50  0000 C CNN
 F 2 "Resistor_SMD:R_0805_2012Metric" H 9900 5300 50  0001 C CNN
 F 3 "~" H 9900 5300 50  0001 C CNN
@@
 P 9200 4100
 F 0 "C45" H 9292 4146 50  0000 L CNN
-F 1 "100p" H 9292 4055 50  0000 L CNN
+F 1 "DNP" H 9292 4055 50  0000 L CNN
 F 2 "Capacitor_SMD:C_0402_1005Metric" H 9200 4100 50  0001 C CNN
 F 3 "~" H 9200 4100 50  0001 C CNN
@@
 P 9200 2250
 F 0 "C44" H 9292 2296 50  0000 L CNN
-F 1 "100p" H 9292 2205 50  0000 L CNN
+F 1 "DNP" H 9292 2205 50  0000 L CNN
 F 2 "Capacitor_SMD:C_0402_1005Metric" H 9200 2250 50  0001 C CNN
 F 3 "~" H 9200 2250 50  0001 C CNN
@@
 L Device:C_Small C43
 U 1 1 5DE96B1D
-P 1150 5750
-F 0 "C43" H 1242 5796 50  0000 L CNN
-F 1 "100n" H 1242 5705 50  0000 L CNN
-F 2 "Capacitor_SMD:C_0603_1608Metric" H 1150 5750 50  0001 C CNN
-F 3 "~" H 1150 5750 50  0001 C CNN
-	1    1150 5750
+P 3000 5700
+F 0 "C43" H 3092 5746 50  0000 L CNN
+F 1 "100n" H 3092 5655 50  0000 L CNN
+F 2 "Capacitor_SMD:C_0603_1608Metric" H 3000 5700 50  0001 C CNN
+F 3 "~" H 3000 5700 50  0001 C CNN
+	1    3000 5700
 	1    0    0    -1
 $EndComp
@@
 L power:GND #PWR0202
 U 1 1 5DE96B23
-P 1150 5850
-F 0 "#PWR0202" H 1150 5600 50  0001 C CNN
-F 1 "GND" H 1155 5677 50  0000 C CNN
-F 2 "" H 1150 5850 50  0001 C CNN
-F 3 "" H 1150 5850 50  0001 C CNN
-	1    1150 5850
+P 3000 5800
+F 0 "#PWR0202" H 3000 5550 50  0001 C CNN
+F 1 "GND" H 3005 5627 50  0000 C CNN
+F 2 "" H 3000 5800 50  0001 C CNN
+F 3 "" H 3000 5800 50  0001 C CNN
+	1    3000 5800
 	1    0    0    -1
 $EndComp
@@
 L Device:C_Small C46
 U 1 1 5DEA0744
-P 2200 5750
-F 0 "C46" H 2292 5796 50  0000 L CNN
-F 1 "100n" H 2292 5705 50  0000 L CNN
-F 2 "Capacitor_SMD:C_0603_1608Metric" H 2200 5750 50  0001 C CNN
-F 3 "~" H 2200 5750 50  0001 C CNN
-	1    2200 5750
+P 4050 5700
+F 0 "C46" H 4142 5746 50  0000 L CNN
+F 1 "100n" H 4142 5655 50  0000 L CNN
+F 2 "Capacitor_SMD:C_0603_1608Metric" H 4050 5700 50  0001 C CNN
+F 3 "~" H 4050 5700 50  0001 C CNN
+	1    4050 5700
 	1    0    0    -1
 $EndComp
@@
 L power:GND #PWR0203
 U 1 1 5DEA074A
-P 2200 5850
-F 0 "#PWR0203" H 2200 5600 50  0001 C CNN
-F 1 "GND" H 2205 5677 50  0000 C CNN
-F 2 "" H 2200 5850 50  0001 C CNN
-F 3 "" H 2200 5850 50  0001 C CNN
-	1    2200 5850
-	1    0    0    -1
-$EndComp
-Wire Wire Line
-	1150 5550 1150 5650
-Wire Wire Line
-	1150 5650 1400 5650
-Connection ~ 1150 5650
-Wire Wire Line
-	2000 5650 2200 5650
+P 4050 5800
+F 0 "#PWR0203" H 4050 5550 50  0001 C CNN
+F 1 "GND" H 4055 5627 50  0000 C CNN
+F 2 "" H 4050 5800 50  0001 C CNN
+F 3 "" H 4050 5800 50  0001 C CNN
+	1    4050 5800
+	1    0    0    -1
+$EndComp
+Wire Wire Line
+	3000 5500 3000 5600
+Wire Wire Line
+	3000 5600 3250 5600
+Connection ~ 3000 5600
+Wire Wire Line
+	3850 5600 4050 5600
 $Comp
 L power:GND #PWR0205
 U 1 1 5DED29D4
-P 1700 5950
-F 0 "#PWR0205" H 1700 5700 50  0001 C CNN
-F 1 "GND" H 1705 5777 50  0000 C CNN
-F 2 "" H 1700 5950 50  0001 C CNN
-F 3 "" H 1700 5950 50  0001 C CNN
-	1    1700 5950
+P 3550 5900
+F 0 "#PWR0205" H 3550 5650 50  0001 C CNN
+F 1 "GND" H 3555 5727 50  0000 C CNN
+F 2 "" H 3550 5900 50  0001 C CNN
+F 3 "" H 3550 5900 50  0001 C CNN
+	1    3550 5900
 	1    0    0    -1
 $EndComp
@@
 L power:+3.3V #PWR0206
 U 1 1 5DEE1B69
-P 2200 5600
-F 0 "#PWR0206" H 2200 5450 50  0001 C CNN
-F 1 "+3.3V" H 2215 5773 50  0000 C CNN
-F 2 "" H 2200 5600 50  0001 C CNN
-F 3 "" H 2200 5600 50  0001 C CNN
-	1    2200 5600
-	1    0    0    -1
-$EndComp
-Wire Wire Line
-	2200 5650 2200 5600
-Connection ~ 2200 5650
+P 4050 5550
+F 0 "#PWR0206" H 4050 5400 50  0001 C CNN
+F 1 "+3.3V" H 4065 5723 50  0000 C CNN
+F 2 "" H 4050 5550 50  0001 C CNN
+F 3 "" H 4050 5550 50  0001 C CNN
+	1    4050 5550
+	1    0    0    -1
+$EndComp
+Wire Wire Line
+	4050 5600 4050 5550
+Connection ~ 4050 5600
 Text GLabel 3700 3650 2    50   Input ~ 0
 GPIO_BEMF
@@
 P 1000 2750
 F 0 "Y1" V 1046 2506 50  0000 R CNN
-F 1 "8Mhz" V 955 2506 50  0000 R CNN
+F 1 "8Mhz" V 900 2500 50  0000 R CNN
 F 2 "Crystal:Crystal_SMD_3225-4Pin_3.2x2.5mm" H 1000 2750 50  0001 C CNN
 F 3 "~" H 1000 2750 50  0001 C CNN
@@
 U 1 1 5DF08F24
 P 10450 1100
-F 0 "R18" V 10346 1100 50  0000 C CNN
-F 1 "1" V 10255 1100 50  0000 C CNN
+F 0 "R18" H 10509 1146 50  0000 L CNN
+F 1 "1" H 10509 1055 50  0000 L CNN
 F 2 "Resistor_SMD:R_0603_1608Metric" H 10450 1100 50  0001 C CNN
 F 3 "~" H 10450 1100 50  0001 C CNN
@@
 U 1 1 5DF50507
 P 10450 2950
-F 0 "R22" V 10346 2950 50  0000 C CNN
-F 1 "1" V 10255 2950 50  0000 C CNN
+F 0 "R22" H 10509 2996 50  0000 L CNN
+F 1 "1" H 10509 2905 50  0000 L CNN
 F 2 "Resistor_SMD:R_0603_1608Metric" H 10450 2950 50  0001 C CNN
 F 3 "~" H 10450 2950 50  0001 C CNN
@@
 U 1 1 5DF690C9
 P 10450 4800
-F 0 "R43" V 10346 4800 50  0000 C CNN
-F 1 "1" V 10255 4800 50  0000 C CNN
+F 0 "R43" H 10509 4846 50  0000 L CNN
+F 1 "1" H 10509 4755 50  0000 L CNN
 F 2 "Resistor_SMD:R_0603_1608Metric" H 10450 4800 50  0001 C CNN
 F 3 "~" H 10450 4800 50  0001 C CNN
@@
 L Regulator_Linear:AP2204R-3.3 U12
 U 1 1 5E17031B
-P 1700 5650
-F 0 "U12" H 1700 5892 50  0000 C CNN
-F 1 "AP2204R-3.3" H 1700 5801 50  0000 C CNN
-F 2 "Package_TO_SOT_SMD:SOT-89-3" H 1700 5875 50  0001 C CNN
-F 3 "https://www.diodes.com/assets/Datasheets/AP2204.pdf" H 1700 5650 50  0001 C CNN
-	1    1700 5650
+P 3550 5600
+F 0 "U12" H 3550 5842 50  0000 C CNN
+F 1 "AP2204R-3.3" H 3550 5751 50  0000 C CNN
+F 2 "Package_TO_SOT_SMD:SOT-89-3" H 3550 5825 50  0001 C CNN
+F 3 "https://www.diodes.com/assets/Datasheets/AP2204.pdf" H 3550 5600 50  0001 C CNN
+	1    3550 5600
 	1    0    0    -1
 $EndComp
@@
 L power:+5V #PWR0204
 U 1 1 5DFAD6AC
-P 1150 5550
-F 0 "#PWR0204" H 1150 5400 50  0001 C CNN
-F 1 "+5V" H 1165 5723 50  0000 C CNN
-F 2 "" H 1150 5550 50  0001 C CNN
-F 3 "" H 1150 5550 50  0001 C CNN
-	1    1150 5550
-	1    0    0    -1
-$EndComp
+P 3000 5500
+F 0 "#PWR0204" H 3000 5350 50  0001 C CNN
+F 1 "+5V" H 3015 5673 50  0000 C CNN
+F 2 "" H 3000 5500 50  0001 C CNN
+F 3 "" H 3000 5500 50  0001 C CNN
+	1    3000 5500
+	1    0    0    -1
+$EndComp
